File: packages/power/buck/tps62933drlr_3v3_ti_c3200405/layouts/example/example.kicad_pcb (KiCad board)
At the start: 2 copper layers, 11 parts

Commit message: Update TPS62933 buck passives and prune parts
Parts:
- C1, C4: value 0F -> 100nF; footprint Samsung_Electro_Mechanics_CL05B104KB54PNC:C0402 -> Murata_Electronics_GRM155R71H104KE14D:C0402
- C2, C3: value 0F -> 10µF; footprint Samsung_Electro_Mechanics_CL31B106KBHNNNE:C1206 -> Murata_Electronics_GRM31CR61H106KA12L:C1206
- C5, C6: value 0F -> 22µF; footprint Samsung_Electro_Mechanics_CL31A226KAHNNNE:C1206 -> Murata_Electronics_GRM31CR61E226KE15L:C1206
- C7: value 0F -> 33nF; footprint Samsung_Electro_Mechanics_CL05B333KB5VPNC:C0402 -> Murata_Electronics_GRM155R71H333KE14D:C0402
- L1: value L 0H -> L 2.2µH
- R1: value 10200Ω -> 10kΩ; footprint UNI_ROYAL_0402WGF1022TCE:R0402 -> YAGEO_RC0402FR_0710KL:R0402
- R2: value 31600Ω -> 31.6kΩ; footprint UNI_ROYAL_0402WGF3162TCE:R0402 -> YAGEO_RC0402FR_0731K6L:R0402
