File: packages/power/power_mux/tps2121ruxr_20v_4a_ti/layouts/example/example.kicad_pcb (KiCad board)
At the start: 2 copper layers, 13 parts

Commit message: Finish removing net-name overrides from reusable packages
This completes the package-level override cleanup by deleting the remaining
`override_net_name` assignments from the library's reusable package modules and
rebuilding their checked-in layouts so generated net metadata matches source.
The package interfaces stay the same; only the forced net naming was removed so
these modules compose cleanly when imported into downstream designs.

Constraint: The library must stay reusable and avoid imposed internal net names leaking into consuming designs
Constraint: Each changed package must still verify with the repo's Atopile workflow after layout regeneration
Rejected: Stop after the battery frontend cleanup | leaves the same composition hazard in other packages
Rejected: Remove override lines without rebuilding layouts | would leave stale generated PCB net names checked into the repo
Confidence: high
Scope-risk: moderate
Reversibility: clean
Directive: Do not reintroduce `override_net_name` in reusable package modules unless a package is intentionally design-specific
Tested: `uv tool run --from atopile==0.15.4 ato --non-interactive build` in each affected package directory (stm32g0b1kbu6_st, mcp2518fdt_e_sl_microchip, tcan3413ddfr_ti, raspberry_pi_hat_socket_zhouri, tps56637rpar_5v1_5a_ti, tps62933drlr_3v3_ti, bq25756rrvr_4s_2a_ti, tps2121ruxr_20v_4a_ti, tps25730drefr_20v_3a_ti)
Not-tested: Downstream consumer projects that may have been depending on the old forced net names in generated layouts
Connections:
- net FALLBACK_SEL renamed 1
- net GND renamed lv
- net HIGH_PRIORITY renamed high_priority-hv
- net LOW_PRIORITY renamed hv
- net OUT renamed out-hv
- net PRIORITY_SEL renamed mux-1
Changed lines of the file:
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@@
 		)
 	)
-	(net 1 "FALLBACK_SEL")
-	(net 2 "OUT")
+	(net 1 "1")
+	(net 2 "out-hv")
 	(net 3 "ILM")
-	(net 4 "GND")
-	(net 5 "LOW_PRIORITY")
-	(net 6 "HIGH_PRIORITY")
+	(net 4 "lv")
+	(net 5 "hv")
+	(net 6 "high_priority-hv")
 	(net 7 "ST")
-	(net 8 "PRIORITY_SEL")
+	(net 8 "mux-1")
 	(net 9 "SS")
 	(footprint "Texas_Instruments_TPS2121RUXR:TPS2121RUXR"
@@
 			(size 0.4 1.05)
 			(layers "F.Cu" "F.Paste" "F.Mask")
-			(net 2 "OUT")
+			(net 2 "out-hv")
 		)
 		(pad "2" smd rect
@@
 			(size 0.4 1.05)
 			(layers "F.Cu" "F.Paste" "F.Mask")
-			(net 5 "LOW_PRIORITY")
+			(net 5 "hv")
 		)
 		(pad "3" smd rect
@@
 			(size 0.2 0.6)
 			(layers "F.Cu" "F.Paste" "F.Mask")
-			(net 1 "FALLBACK_SEL")
+			(net 1 "1")
 		)
 		(pad "4" smd rect
@@
 			(size 0.2 0.6)
 			(layers "F.Cu" "F.Paste" "F.Mask")
-			(net 4 "GND")
+			(net 4 "lv")
 		)
 		(pad "5" smd rect
@@
 			(size 0.2 0.6)
 			(layers "F.Cu" "F.Paste" "F.Mask")
-			(net 4 "GND")
+			(net 4 "lv")
 		)
 		(pad "6" smd rect
@@
 			(size 0.2 0.6)
 			(layers "F.Cu" "F.Paste" "F.Mask")
-			(net 8 "PRIORITY_SEL")
+			(net 8 "mux-1")
 		)
 		(pad "7" smd rect
@@
 			(size 0.4 1.05)
 			(layers "F.Cu" "F.Paste" "F.Mask")
-			(net 6 "HIGH_PRIORITY")
+			(net 6 "high_priority-hv")
 		)
 		(pad "8" smd rect
@@
 			(size 0.4 1.05)
 			(layers "F.Cu" "F.Paste" "F.Mask")
-			(net 2 "OUT")
+			(net 2 "out-hv")
 		)
 		(pad "9" smd rect
@@
 			(size 0.2 0.6)
 			(layers "F.Cu" "F.Paste" "F.Mask")
-			(net 4 "GND")
+			(net 4 "lv")
 		)
 	)
@@
 			(size 1.49 1.73)
 			(layers "F.Cu" "F.Paste" "F.Mask")
-			(net 4 "GND")
+			(net 4 "lv")
 		)
 		(pad "1" smd rect
@@
 			(size 1.49 1.73)
 			(layers "F.Cu" "F.Paste" "F.Mask")
-			(net 6 "HIGH_PRIORITY")
+			(net 6 "high_priority-hv")
 		)
 		(embedded_fonts no)
@@
 			(size 0.5 0.54)
 			(layers "F.Cu" "F.Paste" "F.Mask")
-			(net 4 "GND")
+			(net 4 "lv")
 		)
 		(pad "1" smd rect
@@
 			(size 0.5 0.54)
 			(layers "F.Cu" "F.Paste" "F.Mask")
-			(net 6 "HIGH_PRIORITY")
+			(net 6 "high_priority-hv")
 		)
 		(embedded_fonts no)
@@
 			(size 1.49 1.73)
 			(layers "F.Cu" "F.Paste" "F.Mask")
-			(net 4 "GND")
+			(net 4 "lv")
 		)
 		(pad "1" smd rect
@@
 			(size 1.49 1.73)
 			(layers "F.Cu" "F.Paste" "F.Mask")
-			(net 5 "LOW_PRIORITY")
+			(net 5 "hv")
 		)
 		(embedded_fonts no)
@@
 			(size 0.5 0.54)
 			(layers "F.Cu" "F.Paste" "F.Mask")
-			(net 4 "GND")
+			(net 4 "lv")
 		)
 		(pad "1" smd rect
@@
 			(size 0.5 0.54)
 			(layers "F.Cu" "F.Paste" "F.Mask")
-			(net 5 "LOW_PRIORITY")
+			(net 5 "hv")
 		)
 		(embedded_fonts no)
@@
 			(size 1.49 1.73)
 			(layers "F.Cu" "F.Paste" "F.Mask")
-			(net 4 "GND")
+			(net 4 "lv")
 		)
 		(pad "1" smd rect
@@
 			(size 1.49 1.73)
 			(layers "F.Cu" "F.Paste" "F.Mask")
-			(net 2 "OUT")
+			(net 2 "out-hv")
 		)
 		(embedded_fonts no)
@@
 			(size 0.5 0.54)
 			(layers "F.Cu" "F.Paste" "F.Mask")
-			(net 4 "GND")
+			(net 4 "lv")
 		)
 		(pad "1" smd rect
@@
 			(size 0.5 0.54)
 			(layers "F.Cu" "F.Paste" "F.Mask")
-			(net 2 "OUT")
+			(net 2 "out-hv")
 		)
 		(embedded_fonts no)
@@
 			(size 0.57 0.54)
 			(layers "F.Cu" "F.Paste" "F.Mask")
-			(net 8 "PRIORITY_SEL")
+			(net 8 "mux-1")
 		)
 		(pad "1" smd rect
@@
 			(size 0.57 0.54)
 			(layers "F.Cu" "F.Paste" "F.Mask")
-			(net 6 "HIGH_PRIORITY")
+			(net 6 "high_priority-hv")
 		)
 		(embedded_fonts no)
@@
 			(size 0.57 0.54)
 			(layers "F.Cu" "F.Paste" "F.Mask")
-			(net 4 "GND")
+			(net 4 "lv")
 		)
 		(pad "1" smd rect
@@
 			(size 0.57 0.54)
 			(layers "F.Cu" "F.Paste" "F.Mask")
-			(net 8 "PRIORITY_SEL")
+			(net 8 "mux-1")
 		)
 		(embedded_fonts no)
@@
 			(size 0.57 0.54)
 			(layers "F.Cu" "F.Paste" "F.Mask")
-			(net 1 "FALLBACK_SEL")
+			(net 1 "1")
 		)
 		(pad "1" smd rect
@@
 			(size 0.57 0.54)
 			(layers "F.Cu" "F.Paste" "F.Mask")
-			(net 5 "LOW_PRIORITY")
+			(net 5 "hv")
 		)
 		(embedded_fonts no)
@@
 			(size 0.57 0.54)
 			(layers "F.Cu" "F.Paste" "F.Mask")
-			(net 4 "GND")
+			(net 4 "lv")
 		)
 		(pad "1" smd rect
@@
 			(size 0.57 0.54)
 			(layers "F.Cu" "F.Paste" "F.Mask")
-			(net 1 "FALLBACK_SEL")
+			(net 1 "1")
 		)
 		(embedded_fonts no)
@@
 			(size 0.57 0.54)
 			(layers "F.Cu" "F.Paste" "F.Mask")
-			(net 4 "GND")
+			(net 4 "lv")
 		)
 		(pad "1" smd rect
@@
 			(size 0.5 0.54)
 			(layers "F.Cu" "F.Paste" "F.Mask")
-			(net 4 "GND")
+			(net 4 "lv")
 		)
 		(pad "1" smd rect

Commit message: Make package schematics more readable and align passive choices with repo guidance
This pass improves the human-facing quality of the package library.
Explicit local capacitor/resistor parts now carry short descriptive
comments at the point of use, the MCP2518FD package swaps its 1uF bulk
capacitor to a 0603 part to match the current sizing rule, and several
packages add better net-name overrides for exposed and important internal
signals.

Constraint: Repo guidance now prefers explicit local parts and expects readable schematic net names
Constraint: Passive sizing should follow the current MLCC package rule unless a justified exception is needed
Rejected: Keep part instances comment-free | explicit local part names are not readable enough by themselves
Rejected: Leave the MCP2518FD 1uF bulk cap in 0402 | conflicts with the current 1uF-10uF 0603 guidance
Confidence: medium
Scope-risk: moderate
Reversibility: clean
Directive: When instantiating explicit local resistor/capacitor parts, include a short readable comment with the key value/package characteristics unless the name is already obviously human-readable
Tested:  passed for stm32g0b1kbu6_st, mcp2518fdt_e_sl_microchip, tcan3413ddfr_ti, raspberry_pi_hat_socket_zhouri, bq40z50rsmr_r2_4s_3a_ti, tps56637rpar_5v1_5a_ti, tps62933drlr_3v3_ti, bq25756rrvr_4s_2a_ti, tps2121ruxr_20v_4a_ti, and tps25730drefr_20v_3a_ti
Not-tested: Complete elimination of all internal autogenerated net labels in every package; some deep internal nets may still remain tool-driven
Connections:
- net 1 renamed FALLBACK_SEL
- net high_priority-hv renamed HIGH_PRIORITY
- net hv renamed LOW_PRIORITY
- net lv renamed GND
- net mux-1 renamed PRIORITY_SEL
- net out-hv renamed OUT
Changed lines of the file:
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@@
 		)
 	)
-	(net 1 "1")
-	(net 2 "out-hv")
+	(net 1 "FALLBACK_SEL")
+	(net 2 "OUT")
 	(net 3 "ILM")
-	(net 4 "lv")
-	(net 5 "hv")
-	(net 6 "high_priority-hv")
+	(net 4 "GND")
+	(net 5 "LOW_PRIORITY")
+	(net 6 "HIGH_PRIORITY")
 	(net 7 "ST")
-	(net 8 "mux-1")
+	(net 8 "PRIORITY_SEL")
 	(net 9 "SS")
 	(footprint "Texas_Instruments_TPS2121RUXR:TPS2121RUXR"
@@
 			(size 0.4 1.05)
 			(layers "F.Cu" "F.Paste" "F.Mask")
-			(net 2 "out-hv")
+			(net 2 "OUT")
 		)
 		(pad "2" smd rect
@@
 			(size 0.4 1.05)
 			(layers "F.Cu" "F.Paste" "F.Mask")
-			(net 5 "hv")
+			(net 5 "LOW_PRIORITY")
 		)
 		(pad "3" smd rect
@@
 			(size 0.2 0.6)
 			(layers "F.Cu" "F.Paste" "F.Mask")
-			(net 1 "1")
+			(net 1 "FALLBACK_SEL")
 		)
 		(pad "4" smd rect
@@
 			(size 0.2 0.6)
 			(layers "F.Cu" "F.Paste" "F.Mask")
-			(net 4 "lv")
+			(net 4 "GND")
 		)
 		(pad "5" smd rect
@@
 			(size 0.2 0.6)
 			(layers "F.Cu" "F.Paste" "F.Mask")
-			(net 4 "lv")
+			(net 4 "GND")
 		)
 		(pad "6" smd rect
@@
 			(size 0.2 0.6)
 			(layers "F.Cu" "F.Paste" "F.Mask")
-			(net 8 "mux-1")
+			(net 8 "PRIORITY_SEL")
 		)
 		(pad "7" smd rect
@@
 			(size 0.4 1.05)
 			(layers "F.Cu" "F.Paste" "F.Mask")
-			(net 6 "high_priority-hv")
+			(net 6 "HIGH_PRIORITY")
 		)
 		(pad "8" smd rect
@@
 			(size 0.4 1.05)
 			(layers "F.Cu" "F.Paste" "F.Mask")
-			(net 2 "out-hv")
+			(net 2 "OUT")
 		)
 		(pad "9" smd rect
@@
 			(size 0.2 0.6)
 			(layers "F.Cu" "F.Paste" "F.Mask")
-			(net 4 "lv")
+			(net 4 "GND")
 		)
 	)
@@
 			(size 1.49 1.73)
 			(layers "F.Cu" "F.Paste" "F.Mask")
-			(net 4 "lv")
+			(net 4 "GND")
 		)
 		(pad "1" smd rect
@@
 			(size 1.49 1.73)
 			(layers "F.Cu" "F.Paste" "F.Mask")
-			(net 6 "high_priority-hv")
+			(net 6 "HIGH_PRIORITY")
 		)
 		(embedded_fonts no)
@@
 			(size 0.5 0.54)
 			(layers "F.Cu" "F.Paste" "F.Mask")
-			(net 4 "lv")
+			(net 4 "GND")
 		)
 		(pad "1" smd rect
@@
 			(size 0.5 0.54)
 			(layers "F.Cu" "F.Paste" "F.Mask")
-			(net 6 "high_priority-hv")
+			(net 6 "HIGH_PRIORITY")
 		)
 		(embedded_fonts no)
@@
 			(size 1.49 1.73)
 			(layers "F.Cu" "F.Paste" "F.Mask")
-			(net 4 "lv")
+			(net 4 "GND")
 		)
 		(pad "1" smd rect
@@
 			(size 1.49 1.73)
 			(layers "F.Cu" "F.Paste" "F.Mask")
-			(net 5 "hv")
+			(net 5 "LOW_PRIORITY")
 		)
 		(embedded_fonts no)
@@
 			(size 0.5 0.54)
 			(layers "F.Cu" "F.Paste" "F.Mask")
-			(net 4 "lv")
+			(net 4 "GND")
 		)
 		(pad "1" smd rect
@@
 			(size 0.5 0.54)
 			(layers "F.Cu" "F.Paste" "F.Mask")
-			(net 5 "hv")
+			(net 5 "LOW_PRIORITY")
 		)
 		(embedded_fonts no)
@@
 			(size 1.49 1.73)
 			(layers "F.Cu" "F.Paste" "F.Mask")
-			(net 4 "lv")
+			(net 4 "GND")
 		)
 		(pad "1" smd rect
@@
 			(size 1.49 1.73)
 			(layers "F.Cu" "F.Paste" "F.Mask")
-			(net 2 "out-hv")
+			(net 2 "OUT")
 		)
 		(embedded_fonts no)
@@
 			(size 0.5 0.54)
 			(layers "F.Cu" "F.Paste" "F.Mask")
-			(net 4 "lv")
+			(net 4 "GND")
 		)
 		(pad "1" smd rect
@@
 			(size 0.5 0.54)
 			(layers "F.Cu" "F.Paste" "F.Mask")
-			(net 2 "out-hv")
+			(net 2 "OUT")
 		)
 		(embedded_fonts no)
@@
 			(size 0.57 0.54)
 			(layers "F.Cu" "F.Paste" "F.Mask")
-			(net 8 "mux-1")
+			(net 8 "PRIORITY_SEL")
 		)
 		(pad "1" smd rect
@@
 			(size 0.57 0.54)
 			(layers "F.Cu" "F.Paste" "F.Mask")
-			(net 6 "high_priority-hv")
+			(net 6 "HIGH_PRIORITY")
 		)
 		(embedded_fonts no)
@@
 			(size 0.57 0.54)
 			(layers "F.Cu" "F.Paste" "F.Mask")
-			(net 4 "lv")
+			(net 4 "GND")
 		)
 		(pad "1" smd rect
@@
 			(size 0.57 0.54)
 			(layers "F.Cu" "F.Paste" "F.Mask")
-			(net 8 "mux-1")
+			(net 8 "PRIORITY_SEL")
 		)
 		(embedded_fonts no)
@@
 			(size 0.57 0.54)
 			(layers "F.Cu" "F.Paste" "F.Mask")
-			(net 1 "1")
+			(net 1 "FALLBACK_SEL")
 		)
 		(pad "1" smd rect
@@
 			(size 0.57 0.54)
 			(layers "F.Cu" "F.Paste" "F.Mask")
-			(net 5 "hv")
+			(net 5 "LOW_PRIORITY")
 		)
 		(embedded_fonts no)
@@
 			(size 0.57 0.54)
 			(layers "F.Cu" "F.Paste" "F.Mask")
-			(net 4 "lv")
+			(net 4 "GND")
 		)
 		(pad "1" smd rect
@@
 			(size 0.57 0.54)
 			(layers "F.Cu" "F.Paste" "F.Mask")
-			(net 1 "1")
+			(net 1 "FALLBACK_SEL")
 		)
 		(embedded_fonts no)
@@
 			(size 0.57 0.54)
 			(layers "F.Cu" "F.Paste" "F.Mask")
-			(net 4 "lv")
+			(net 4 "GND")
 		)
 		(pad "1" smd rect
@@
 			(size 0.5 0.54)
 			(layers "F.Cu" "F.Paste" "F.Mask")
-			(net 4 "lv")
+			(net 4 "GND")
 		)
 		(pad "1" smd rect
