File: packages/embedded/mcu/stm32g0b1kbu6_st/layouts/example/example.kicad_pcb (KiCad board)
At the start: 2 copper layers, 5 parts

Commit message: Make package builds deterministic by wiring explicit local parts
The remaining packages now reference package-local concrete passives,
inductors, and other small parts directly instead of relying on generic
part-picker resolution. This aligns the source with the local
assets and removes the flaky live EasyEDA lookup path that was blocking
verification.

Constraint: Builds must not depend on unstable live part-picking when local package assets already exist
Constraint: Package-local parts remain the ownership boundary; no shared global part store was introduced
Rejected: Keep generic passives as the default style | repeated verification failures from upstream EasyEDA API instability
Rejected: Add ad hoc offline hacks around ato part-picking | weaker than making the package source deterministic
Confidence: high
Scope-risk: moderate
Reversibility: clean
Directive: For packages that already own generated local parts, instantiate those part modules directly and avoid generic passive declarations unless there is a strong reason not to
Tested:  passed for stm32g0b1kbu6_st, mcp2518fdt_e_sl_microchip, tcan3413ddfr_ti, raspberry_pi_hat_socket_zhouri, bq40z50rsmr_r2_4s_3a_ti, tps56637rpar_5v1_5a_ti, tps62933drlr_3v3_ti, bq25756rrvr_4s_2a_ti, tps2121ruxr_20v_4a_ti, and tps25730drefr_20v_3a_ti
Not-tested: Cross-package downstream integration beyond each package's default/example build
Parts:
- C1, C3: value 100nF ±10% -> (none)
- C2: value 4.7µF ±10% -> (none)
- R1: value 10kΩ ±1% -> (none)
Connections:
- C1 pad 1: hv -> PF2_NRST
- C2 pad 1: supply_bypass-power-hv -> hv
- C3 pad 1: supply_bypass-power-hv -> hv
- U1 pad 4: supply_bypass-power-hv -> hv
- U1 pad 6: hv -> PF2_NRST
Changed lines of the file:
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@@
 	(net 26 "PB8")
 	(net 27 "lv")
-	(net 28 "hv")
+	(net 28 "PF2_NRST")
 	(net 29 "PA0")
 	(net 30 "PA1")
 	(net 31 "PA2")
-	(net 32 "supply_bypass-power-hv")
+	(net 32 "hv")
 	(footprint "STMicroelectronics_STM32G0B1KBU6:QFN-32_L5.0-W5.0-P0.50-TL-EP3.5"
 		(layer "F.Cu")
@@
 			(size 0.8 0.28)
 			(layers "F.Cu" "F.Paste" "F.Mask")
-			(net 32 "supply_bypass-power-hv")
+			(net 32 "hv")
 		)
 		(pad "5" smd oval
@@
 			(size 0.8 0.28)
 			(layers "F.Cu" "F.Paste" "F.Mask")
-			(net 28 "hv")
+			(net 28 "PF2_NRST")
 		)
 		(pad "7" smd oval
@@
 			)
 		)
-		(property "Value" "10kΩ ±1%"
+		(property "Value" ""
 			(at 0 4)
 			(layer "F.Fab")
@@
 			(hide yes)
 		)
-		(property "Datasheet" "https://www.lcsc.com/datasheet/lcsc_datasheet_1811141608_YAGEO-RC0402FR-0710KL_C60490.pdf"
+		(property "Datasheet" "https://www.lcsc.com/datasheet/lcsc_datasheet_2304140030_YAGEO-RC0402FR-0710KL_C60490.pdf"
 			(at 0 0 0)
 			(layer "User.9")
@@
 			)
 		)
-		(property "Value" "100nF ±10%"
+		(property "Value" ""
 			(at 0 4)
 			(layer "F.Fab")
@@
 			(size 0.5 0.54)
 			(layers "F.Cu" "F.Paste" "F.Mask")
-			(net 28 "hv")
+			(net 28 "PF2_NRST")
 		)
 		(embedded_fonts no)
@@
 			)
 		)
-		(property "Value" "100nF ±10%"
+		(property "Value" ""
 			(at 0 4)
 			(layer "F.Fab")
@@
 			(size 0.5 0.54)
 			(layers "F.Cu" "F.Paste" "F.Mask")
-			(net 32 "supply_bypass-power-hv")
+			(net 32 "hv")
 		)
 		(embedded_fonts no)
@@
 			)
 		)
-		(property "Value" "4.7µF ±10%"
+		(property "Value" ""
 			(at 0 4)
 			(layer "F.Fab")
@@
 			(size 0.8 0.9)
 			(layers "F.Cu" "F.Paste" "F.Mask")
-			(net 32 "supply_bypass-power-hv")
+			(net 32 "hv")
 		)
 		(embedded_fonts no)

Commit message: Make package schematics more readable and align passive choices with repo guidance
This pass improves the human-facing quality of the package library.
Explicit local capacitor/resistor parts now carry short descriptive
comments at the point of use, the MCP2518FD package swaps its 1uF bulk
capacitor to a 0603 part to match the current sizing rule, and several
packages add better net-name overrides for exposed and important internal
signals.

Constraint: Repo guidance now prefers explicit local parts and expects readable schematic net names
Constraint: Passive sizing should follow the current MLCC package rule unless a justified exception is needed
Rejected: Keep part instances comment-free | explicit local part names are not readable enough by themselves
Rejected: Leave the MCP2518FD 1uF bulk cap in 0402 | conflicts with the current 1uF-10uF 0603 guidance
Confidence: medium
Scope-risk: moderate
Reversibility: clean
Directive: When instantiating explicit local resistor/capacitor parts, include a short readable comment with the key value/package characteristics unless the name is already obviously human-readable
Tested:  passed for stm32g0b1kbu6_st, mcp2518fdt_e_sl_microchip, tcan3413ddfr_ti, raspberry_pi_hat_socket_zhouri, bq40z50rsmr_r2_4s_3a_ti, tps56637rpar_5v1_5a_ti, tps62933drlr_3v3_ti, bq25756rrvr_4s_2a_ti, tps2121ruxr_20v_4a_ti, and tps25730drefr_20v_3a_ti
Not-tested: Complete elimination of all internal autogenerated net labels in every package; some deep internal nets may still remain tool-driven
Connections:
- net hv renamed +3.3V
- net lv renamed GND
Changed lines of the file:
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@@
 	(net 25 "PB7")
 	(net 26 "PB8")
-	(net 27 "lv")
+	(net 27 "GND")
 	(net 28 "PF2_NRST")
 	(net 29 "PA0")
 	(net 30 "PA1")
 	(net 31 "PA2")
-	(net 32 "hv")
+	(net 32 "+3.3V")
 	(footprint "STMicroelectronics_STM32G0B1KBU6:QFN-32_L5.0-W5.0-P0.50-TL-EP3.5"
 		(layer "F.Cu")
@@
 			(size 3.5 3.5)
 			(layers "F.Cu" "F.Paste" "F.Mask")
-			(net 27 "lv")
+			(net 27 "GND")
 		)
 		(pad "1" smd oval
@@
 			(size 0.8 0.28)
 			(layers "F.Cu" "F.Paste" "F.Mask")
-			(net 32 "hv")
+			(net 32 "+3.3V")
 		)
 		(pad "5" smd oval
@@
 			(size 0.8 0.28)
 			(layers "F.Cu" "F.Paste" "F.Mask")
-			(net 27 "lv")
+			(net 27 "GND")
 		)
 		(pad "6" smd oval
@@
 			(size 0.57 0.54)
 			(layers "F.Cu" "F.Paste" "F.Mask")
-			(net 27 "lv")
+			(net 27 "GND")
 		)
 		(pad "1" smd rect
@@
 			(size 0.5 0.54)
 			(layers "F.Cu" "F.Paste" "F.Mask")
-			(net 27 "lv")
+			(net 27 "GND")
 		)
 		(pad "1" smd rect
@@
 			(size 0.5 0.54)
 			(layers "F.Cu" "F.Paste" "F.Mask")
-			(net 27 "lv")
+			(net 27 "GND")
 		)
 		(pad "1" smd rect
@@
 			(size 0.5 0.54)
 			(layers "F.Cu" "F.Paste" "F.Mask")
-			(net 32 "hv")
+			(net 32 "+3.3V")
 		)
 		(embedded_fonts no)
@@
 			(size 0.8 0.9)
 			(layers "F.Cu" "F.Paste" "F.Mask")
-			(net 27 "lv")
+			(net 27 "GND")
 		)
 		(pad "1" smd rect
@@
 			(size 0.8 0.9)
 			(layers "F.Cu" "F.Paste" "F.Mask")
-			(net 32 "hv")
+			(net 32 "+3.3V")
 		)
 		(embedded_fonts no)

Commit message: Finish removing net-name overrides from reusable packages
This completes the package-level override cleanup by deleting the remaining
`override_net_name` assignments from the library's reusable package modules and
rebuilding their checked-in layouts so generated net metadata matches source.
The package interfaces stay the same; only the forced net naming was removed so
these modules compose cleanly when imported into downstream designs.

Constraint: The library must stay reusable and avoid imposed internal net names leaking into consuming designs
Constraint: Each changed package must still verify with the repo's Atopile workflow after layout regeneration
Rejected: Stop after the battery frontend cleanup | leaves the same composition hazard in other packages
Rejected: Remove override lines without rebuilding layouts | would leave stale generated PCB net names checked into the repo
Confidence: high
Scope-risk: moderate
Reversibility: clean
Directive: Do not reintroduce `override_net_name` in reusable package modules unless a package is intentionally design-specific
Tested: `uv tool run --from atopile==0.15.4 ato --non-interactive build` in each affected package directory (stm32g0b1kbu6_st, mcp2518fdt_e_sl_microchip, tcan3413ddfr_ti, raspberry_pi_hat_socket_zhouri, tps56637rpar_5v1_5a_ti, tps62933drlr_3v3_ti, bq25756rrvr_4s_2a_ti, tps2121ruxr_20v_4a_ti, tps25730drefr_20v_3a_ti)
Not-tested: Downstream consumer projects that may have been depending on the old forced net names in generated layouts
Connections:
- net +3.3V renamed hv
- net GND renamed lv
Changed lines of the file:
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@@
 	(net 25 "PB7")
 	(net 26 "PB8")
-	(net 27 "GND")
+	(net 27 "lv")
 	(net 28 "PF2_NRST")
 	(net 29 "PA0")
 	(net 30 "PA1")
 	(net 31 "PA2")
-	(net 32 "+3.3V")
+	(net 32 "hv")
 	(footprint "STMicroelectronics_STM32G0B1KBU6:QFN-32_L5.0-W5.0-P0.50-TL-EP3.5"
 		(layer "F.Cu")
@@
 			(size 3.5 3.5)
 			(layers "F.Cu" "F.Paste" "F.Mask")
-			(net 27 "GND")
+			(net 27 "lv")
 		)
 		(pad "1" smd oval
@@
 			(size 0.8 0.28)
 			(layers "F.Cu" "F.Paste" "F.Mask")
-			(net 32 "+3.3V")
+			(net 32 "hv")
 		)
 		(pad "5" smd oval
@@
 			(size 0.8 0.28)
 			(layers "F.Cu" "F.Paste" "F.Mask")
-			(net 27 "GND")
+			(net 27 "lv")
 		)
 		(pad "6" smd oval
@@
 			(size 0.57 0.54)
 			(layers "F.Cu" "F.Paste" "F.Mask")
-			(net 27 "GND")
+			(net 27 "lv")
 		)
 		(pad "1" smd rect
@@
 			(size 0.5 0.54)
 			(layers "F.Cu" "F.Paste" "F.Mask")
-			(net 27 "GND")
+			(net 27 "lv")
 		)
 		(pad "1" smd rect
@@
 			(size 0.5 0.54)
 			(layers "F.Cu" "F.Paste" "F.Mask")
-			(net 27 "GND")
+			(net 27 "lv")
 		)
 		(pad "1" smd rect
@@
 			(size 0.5 0.54)
 			(layers "F.Cu" "F.Paste" "F.Mask")
-			(net 32 "+3.3V")
+			(net 32 "hv")
 		)
 		(embedded_fonts no)
@@
 			(size 0.8 0.9)
 			(layers "F.Cu" "F.Paste" "F.Mask")
-			(net 27 "GND")
+			(net 27 "lv")
 		)
 		(pad "1" smd rect
@@
 			(size 0.8 0.9)
 			(layers "F.Cu" "F.Paste" "F.Mask")
-			(net 32 "+3.3V")
+			(net 32 "hv")
 		)
 		(embedded_fonts no)
