File: packages/interface/connector/raspberry_pi_hat_socket_zhouri/layouts/example/example.kicad_pcb (KiCad board)
At the start: 2 copper layers, 1 part

Commit message: Make package schematics more readable and align passive choices with repo guidance
This pass improves the human-facing quality of the package library.
Explicit local capacitor/resistor parts now carry short descriptive
comments at the point of use, the MCP2518FD package swaps its 1uF bulk
capacitor to a 0603 part to match the current sizing rule, and several
packages add better net-name overrides for exposed and important internal
signals.

Constraint: Repo guidance now prefers explicit local parts and expects readable schematic net names
Constraint: Passive sizing should follow the current MLCC package rule unless a justified exception is needed
Rejected: Keep part instances comment-free | explicit local part names are not readable enough by themselves
Rejected: Leave the MCP2518FD 1uF bulk cap in 0402 | conflicts with the current 1uF-10uF 0603 guidance
Confidence: medium
Scope-risk: moderate
Reversibility: clean
Directive: When instantiating explicit local resistor/capacitor parts, include a short readable comment with the key value/package characteristics unless the name is already obviously human-readable
Tested:  passed for stm32g0b1kbu6_st, mcp2518fdt_e_sl_microchip, tcan3413ddfr_ti, raspberry_pi_hat_socket_zhouri, bq40z50rsmr_r2_4s_3a_ti, tps56637rpar_5v1_5a_ti, tps62933drlr_3v3_ti, bq25756rrvr_4s_2a_ti, tps2121ruxr_20v_4a_ti, and tps25730drefr_20v_3a_ti
Not-tested: Complete elimination of all internal autogenerated net labels in every package; some deep internal nets may still remain tool-driven
Connections:
- net hv renamed +3.3V
- net lv renamed GND
- net power_5v0-hv renamed +5V
Changed lines of the file:
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@@
 	(net 38 "P07_GPIO4_GPCLK0")
 	(net 39 "P08_GPIO14_TXD0")
-	(net 41 "hv")
-	(net 42 "lv")
-	(net 43 "power_5v0-hv")
+	(net 41 "+3.3V")
+	(net 42 "GND")
+	(net 43 "+5V")
 	(footprint "ZHOURI_2_54_2_20:HDR-TH_40P-P2.54-V-F-R2-C20-S2.54"
 		(layer "F.Cu")
@@
 			(drill 0.999998)
 			(layers "*.Cu" "*.Mask")
-			(net 42 "lv")
+			(net 42 "GND")
 		)
 		(pad "38" thru_hole circle
@@
 			(drill 0.999998)
 			(layers "*.Cu" "*.Mask")
-			(net 42 "lv")
+			(net 42 "GND")
 		)
 		(pad "33" thru_hole circle
@@
 			(drill 0.999998)
 			(layers "*.Cu" "*.Mask")
-			(net 42 "lv")
+			(net 42 "GND")
 		)
 		(pad "29" thru_hole circle
@@
 			(drill 0.999998)
 			(layers "*.Cu" "*.Mask")
-			(net 42 "lv")
+			(net 42 "GND")
 		)
 		(pad "24" thru_hole circle
@@
 			(drill 0.999998)
 			(layers "*.Cu" "*.Mask")
-			(net 42 "lv")
+			(net 42 "GND")
 		)
 		(pad "19" thru_hole circle
@@
 			(drill 0.999998)
 			(layers "*.Cu" "*.Mask")
-			(net 41 "hv")
+			(net 41 "+3.3V")
 		)
 		(pad "16" thru_hole circle
@@
 			(drill 0.999998)
 			(layers "*.Cu" "*.Mask")
-			(net 42 "lv")
+			(net 42 "GND")
 		)
 		(pad "13" thru_hole circle
@@
 			(drill 0.999998)
 			(layers "*.Cu" "*.Mask")
-			(net 42 "lv")
+			(net 42 "GND")
 		)
 		(pad "8" thru_hole circle
@@
 			(drill 0.999998)
 			(layers "*.Cu" "*.Mask")
-			(net 42 "lv")
+			(net 42 "GND")
 		)
 		(pad "5" thru_hole circle
@@
 			(drill 0.999998)
 			(layers "*.Cu" "*.Mask")
-			(net 43 "power_5v0-hv")
+			(net 43 "+5V")
 		)
 		(pad "3" thru_hole circle
@@
 			(drill 0.999998)
 			(layers "*.Cu" "*.Mask")
-			(net 43 "power_5v0-hv")
+			(net 43 "+5V")
 		)
 		(pad "1" thru_hole rect
@@
 			(drill 0.999998)
 			(layers "*.Cu" "*.Mask")
-			(net 41 "hv")
+			(net 41 "+3.3V")
 		)
 		(embedded_fonts no)

Commit message: Finish removing net-name overrides from reusable packages
This completes the package-level override cleanup by deleting the remaining
`override_net_name` assignments from the library's reusable package modules and
rebuilding their checked-in layouts so generated net metadata matches source.
The package interfaces stay the same; only the forced net naming was removed so
these modules compose cleanly when imported into downstream designs.

Constraint: The library must stay reusable and avoid imposed internal net names leaking into consuming designs
Constraint: Each changed package must still verify with the repo's Atopile workflow after layout regeneration
Rejected: Stop after the battery frontend cleanup | leaves the same composition hazard in other packages
Rejected: Remove override lines without rebuilding layouts | would leave stale generated PCB net names checked into the repo
Confidence: high
Scope-risk: moderate
Reversibility: clean
Directive: Do not reintroduce `override_net_name` in reusable package modules unless a package is intentionally design-specific
Tested: `uv tool run --from atopile==0.15.4 ato --non-interactive build` in each affected package directory (stm32g0b1kbu6_st, mcp2518fdt_e_sl_microchip, tcan3413ddfr_ti, raspberry_pi_hat_socket_zhouri, tps56637rpar_5v1_5a_ti, tps62933drlr_3v3_ti, bq25756rrvr_4s_2a_ti, tps2121ruxr_20v_4a_ti, tps25730drefr_20v_3a_ti)
Not-tested: Downstream consumer projects that may have been depending on the old forced net names in generated layouts
Connections:
- net +3.3V renamed hv
- net +5V renamed power_5v0-hv
- net GND renamed lv
Changed lines of the file:
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@@
 	(net 38 "P07_GPIO4_GPCLK0")
 	(net 39 "P08_GPIO14_TXD0")
-	(net 41 "+3.3V")
-	(net 42 "GND")
-	(net 43 "+5V")
+	(net 41 "hv")
+	(net 42 "lv")
+	(net 43 "power_5v0-hv")
 	(footprint "ZHOURI_2_54_2_20:HDR-TH_40P-P2.54-V-F-R2-C20-S2.54"
 		(layer "F.Cu")
@@
 			(drill 0.999998)
 			(layers "*.Cu" "*.Mask")
-			(net 42 "GND")
+			(net 42 "lv")
 		)
 		(pad "38" thru_hole circle
@@
 			(drill 0.999998)
 			(layers "*.Cu" "*.Mask")
-			(net 42 "GND")
+			(net 42 "lv")
 		)
 		(pad "33" thru_hole circle
@@
 			(drill 0.999998)
 			(layers "*.Cu" "*.Mask")
-			(net 42 "GND")
+			(net 42 "lv")
 		)
 		(pad "29" thru_hole circle
@@
 			(drill 0.999998)
 			(layers "*.Cu" "*.Mask")
-			(net 42 "GND")
+			(net 42 "lv")
 		)
 		(pad "24" thru_hole circle
@@
 			(drill 0.999998)
 			(layers "*.Cu" "*.Mask")
-			(net 42 "GND")
+			(net 42 "lv")
 		)
 		(pad "19" thru_hole circle
@@
 			(drill 0.999998)
 			(layers "*.Cu" "*.Mask")
-			(net 41 "+3.3V")
+			(net 41 "hv")
 		)
 		(pad "16" thru_hole circle
@@
 			(drill 0.999998)
 			(layers "*.Cu" "*.Mask")
-			(net 42 "GND")
+			(net 42 "lv")
 		)
 		(pad "13" thru_hole circle
@@
 			(drill 0.999998)
 			(layers "*.Cu" "*.Mask")
-			(net 42 "GND")
+			(net 42 "lv")
 		)
 		(pad "8" thru_hole circle
@@
 			(drill 0.999998)
 			(layers "*.Cu" "*.Mask")
-			(net 42 "GND")
+			(net 42 "lv")
 		)
 		(pad "5" thru_hole circle
@@
 			(drill 0.999998)
 			(layers "*.Cu" "*.Mask")
-			(net 43 "+5V")
+			(net 43 "power_5v0-hv")
 		)
 		(pad "3" thru_hole circle
@@
 			(drill 0.999998)
 			(layers "*.Cu" "*.Mask")
-			(net 43 "+5V")
+			(net 43 "power_5v0-hv")
 		)
 		(pad "1" thru_hole rect
@@
 			(drill 0.999998)
 			(layers "*.Cu" "*.Mask")
-			(net 41 "+3.3V")
+			(net 41 "hv")
 		)
 		(embedded_fonts no)
