File: packages/power/buck/tps62933drlr_3v3_ti/layouts/example/example.kicad_pcb (KiCad board)
At the start: 2 copper layers, 11 parts

Commit message: Make package builds deterministic by wiring explicit local parts
The remaining packages now reference package-local concrete passives,
inductors, and other small parts directly instead of relying on generic
part-picker resolution. This aligns the source with the local
assets and removes the flaky live EasyEDA lookup path that was blocking
verification.

Constraint: Builds must not depend on unstable live part-picking when local package assets already exist
Constraint: Package-local parts remain the ownership boundary; no shared global part store was introduced
Rejected: Keep generic passives as the default style | repeated verification failures from upstream EasyEDA API instability
Rejected: Add ad hoc offline hacks around ato part-picking | weaker than making the package source deterministic
Confidence: high
Scope-risk: moderate
Reversibility: clean
Directive: For packages that already own generated local parts, instantiate those part modules directly and avoid generic passive declarations unless there is a strong reason not to
Tested:  passed for stm32g0b1kbu6_st, mcp2518fdt_e_sl_microchip, tcan3413ddfr_ti, raspberry_pi_hat_socket_zhouri, bq40z50rsmr_r2_4s_3a_ti, tps56637rpar_5v1_5a_ti, tps62933drlr_3v3_ti, bq25756rrvr_4s_2a_ti, tps2121ruxr_20v_4a_ti, and tps25730drefr_20v_3a_ti
Not-tested: Cross-package downstream integration beyond each package's default/example build
Parts:
- C1, C4: value 100nF -> (none)
- C2, C3: value 10µF -> (none)
- C5, C6: value 22µF -> (none)
- C7: value 33nF -> (none)
- L1: value L 2.2µH -> (none)
- R1: value 10kΩ -> (none)
- R2: value 31.6kΩ -> (none)
Connections:
- net output_bulk_b-power-hv renamed power_out-hv
- net soft_start_cap-power-hv renamed SS
- C1 pad 1: hv -> BST
- C1 pad 2: lv -> SW
- C2 pad 1: input_bypass-power-hv -> hv
- C2 pad 2: soft_start_cap-power-lv -> lv
- C3 pad 1: input_bypass-power-hv -> hv
- C3 pad 2: soft_start_cap-power-lv -> lv
- C4 pad 1: input_bypass-power-hv -> hv
- C4 pad 2: soft_start_cap-power-lv -> lv
- C5 pad 2: soft_start_cap-power-lv -> lv
- C6 pad 2: soft_start_cap-power-lv -> lv
- C7 pad 2: soft_start_cap-power-lv -> lv
- L1 pad 1: lv -> SW
- R1 pad 2: soft_start_cap-power-lv -> lv
- U1 pad 1: soft_start_cap-power-lv -> lv
- U1 pad 2: input_bypass-power-hv -> hv
- U1 pad 3: input_bypass-power-hv -> hv
- U1 pad 4: soft_start_cap-power-lv -> lv
- U1 pad 5: lv -> SW
- U1 pad 6: hv -> BST
Changed lines of the file:
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@@
 	)
 	(net 0 "")
-	(net 3 "hv")
-	(net 4 "soft_start_cap-power-hv")
+	(net 3 "BST")
+	(net 4 "SS")
 	(net 5 "FB")
-	(net 6 "input_bypass-power-hv")
-	(net 8 "soft_start_cap-power-lv")
-	(net 2 "lv")
-	(net 7 "output_bulk_b-power-hv")
+	(net 6 "hv")
+	(net 8 "lv")
+	(net 2 "SW")
+	(net 7 "power_out-hv")
 	(footprint "Texas_Instruments_TPS62933DRLR:SOT-583-8_L2.1-W1.2-P0.50-LS1.6-BR"
 		(layer "F.Cu")
@@
 			(size 0.28 0.68)
 			(layers "F.Cu" "F.Paste" "F.Mask")
-			(net 4 "soft_start_cap-power-hv")
+			(net 4 "SS")
 		)
 		(pad "6" smd rect
@@
 			(size 0.28 0.68)
 			(layers "F.Cu" "F.Paste" "F.Mask")
-			(net 3 "hv")
+			(net 3 "BST")
 		)
 		(pad "5" smd rect
@@
 			(size 0.28 0.68)
 			(layers "F.Cu" "F.Paste" "F.Mask")
-			(net 2 "lv")
+			(net 2 "SW")
 		)
 		(pad "4" smd rect
@@
 			(size 0.28 0.68)
 			(layers "F.Cu" "F.Paste" "F.Mask")
-			(net 8 "soft_start_cap-power-lv")
+			(net 8 "lv")
 		)
 		(pad "3" smd rect
@@
 			(size 0.28 0.68)
 			(layers "F.Cu" "F.Paste" "F.Mask")
-			(net 6 "input_bypass-power-hv")
+			(net 6 "hv")
 		)
 		(pad "2" smd rect
@@
 			(size 0.28 0.68)
 			(layers "F.Cu" "F.Paste" "F.Mask")
-			(net 6 "input_bypass-power-hv")
+			(net 6 "hv")
 		)
 		(pad "1" smd rect
@@
 			(size 0.28 0.68)
 			(layers "F.Cu" "F.Paste" "F.Mask")
-			(net 8 "soft_start_cap-power-lv")
+			(net 8 "lv")
 		)
 		(embedded_fonts no)
@@
 			)
 		)
-		(property "Value" "100nF"
+		(property "Value" ""
 			(at 0 4)
 			(layer "F.Fab")
@@
 			(size 0.5 0.54)
 			(layers "F.Cu" "F.Paste" "F.Mask")
-			(net 2 "lv")
+			(net 2 "SW")
 		)
 		(pad "1" smd rect
@@
 			(size 0.5 0.54)
 			(layers "F.Cu" "F.Paste" "F.Mask")
-			(net 3 "hv")
+			(net 3 "BST")
 		)
 		(embedded_fonts no)
@@
 			)
 		)
-		(property "Value" "100nF"
+		(property "Value" ""
 			(at 0 4)
 			(layer "F.Fab")
@@
 			(size 0.5 0.54)
 			(layers "F.Cu" "F.Paste" "F.Mask")
-			(net 8 "soft_start_cap-power-lv")
+			(net 8 "lv")
 		)
 		(pad "1" smd rect
@@
 			(size 0.5 0.54)
 			(layers "F.Cu" "F.Paste" "F.Mask")
-			(net 6 "input_bypass-power-hv")
+			(net 6 "hv")
 		)
 		(embedded_fonts no)
@@
 			)
 		)
-		(property "Value" "10kΩ"
+		(property "Value" ""
 			(at 0 4)
 			(layer "F.Fab")
@@
 			(hide yes)
 		)
-		(property "Datasheet" "https://www.lcsc.com/datasheet/lcsc_datasheet_1811141608_YAGEO-RC0402FR-0710KL_C60490.pdf"
+		(property "Datasheet" "https://www.lcsc.com/datasheet/lcsc_datasheet_2304140030_YAGEO-RC0402FR-0710KL_C60490.pdf"
 			(at 0 0 0)
 			(layer "User.9")
@@
 			(size 0.57 0.54)
 			(layers "F.Cu" "F.Paste" "F.Mask")
-			(net 8 "soft_start_cap-power-lv")
+			(net 8 "lv")
 		)
 		(pad "1" smd rect
@@
 			)
 		)
-		(property "Value" "31.6kΩ"
+		(property "Value" ""
 			(at 0 4)
 			(layer "F.Fab")
@@
 			(size 0.57 0.54)
 			(layers "F.Cu" "F.Paste" "F.Mask")
-			(net 7 "output_bulk_b-power-hv")
+			(net 7 "power_out-hv")
 		)
 		(embedded_fonts no)
@@
 			)
 		)
-		(property "Value" "10µF"
+		(property "Value" ""
 			(at 0 4)
 			(layer "F.Fab")
@@
 			(size 1.49 1.73)
 			(layers "F.Cu" "F.Paste" "F.Mask")
-			(net 8 "soft_start_cap-power-lv")
+			(net 8 "lv")
 		)
 		(pad "1" smd rect
@@
 			(size 1.49 1.73)
 			(layers "F.Cu" "F.Paste" "F.Mask")
-			(net 6 "input_bypass-power-hv")
+			(net 6 "hv")
 		)
 		(embedded_fonts no)
@@
 			)
 		)
-		(property "Value" "10µF"
+		(property "Value" ""
 			(at 0 4)
 			(layer "F.Fab")
@@
 			(size 1.49 1.73)
 			(layers "F.Cu" "F.Paste" "F.Mask")
-			(net 8 "soft_start_cap-power-lv")
+			(net 8 "lv")
 		)
 		(pad "1" smd rect
@@
 			(size 1.49 1.73)
 			(layers "F.Cu" "F.Paste" "F.Mask")
-			(net 6 "input_bypass-power-hv")
+			(net 6 "hv")
 		)
 		(embedded_fonts no)
@@
 			)
 		)
-		(property "Value" "22µF"
+		(property "Value" ""
 			(at 0 4)
 			(layer "F.Fab")
@@
 			(size 1.49 1.73)
 			(layers "F.Cu" "F.Paste" "F.Mask")
-			(net 8 "soft_start_cap-power-lv")
+			(net 8 "lv")
 		)
 		(pad "1" smd rect
@@
 			(size 1.49 1.73)
 			(layers "F.Cu" "F.Paste" "F.Mask")
-			(net 7 "output_bulk_b-power-hv")
+			(net 7 "power_out-hv")
 		)
 		(embedded_fonts no)
@@
 			)
 		)
-		(property "Value" "22µF"
+		(property "Value" ""
 			(at 0 4)
 			(layer "F.Fab")
@@
 			(size 1.49 1.73)
 			(layers "F.Cu" "F.Paste" "F.Mask")
-			(net 8 "soft_start_cap-power-lv")
+			(net 8 "lv")
 		)
 		(pad "1" smd rect
@@
 			(size 1.49 1.73)
 			(layers "F.Cu" "F.Paste" "F.Mask")
-			(net 7 "output_bulk_b-power-hv")
+			(net 7 "power_out-hv")
 		)
 		(embedded_fonts no)
@@
 			)
 		)
-		(property "Value" "L 2.2µH"
+		(property "Value" ""
 			(at 0 4)
 			(layer "F.Fab")
@@
 			(hide yes)
 		)
-		(property "Manufacturer" "cjiang (Changjiang Microelectronics Tech)"
+		(property "Manufacturer" "cjiang "
 			(at 0 0 0)
 			(layer "User.9")
@@
 			(size 2.2 0.8)
 			(layers "F.Cu" "F.Paste" "F.Mask")
-			(net 7 "output_bulk_b-power-hv")
+			(net 7 "power_out-hv")
 		)
 		(pad "1" smd rect
@@
 			(size 2.2 0.8)
 			(layers "F.Cu" "F.Paste" "F.Mask")
-			(net 2 "lv")
+			(net 2 "SW")
 		)
 		(embedded_fonts no)
@@
 			)
 		)
-		(property "Value" "33nF"
+		(property "Value" ""
 			(at 0 4)
 			(layer "F.Fab")
@@
 			(size 0.5 0.54)
 			(layers "F.Cu" "F.Paste" "F.Mask")
-			(net 8 "soft_start_cap-power-lv")
+			(net 8 "lv")
 		)
 		(pad "1" smd rect
@@
 			(size 0.5 0.54)
 			(layers "F.Cu" "F.Paste" "F.Mask")
-			(net 4 "soft_start_cap-power-hv")
+			(net 4 "SS")
 		)
 		(embedded_fonts no)

Commit message: Make package schematics more readable and align passive choices with repo guidance
This pass improves the human-facing quality of the package library.
Explicit local capacitor/resistor parts now carry short descriptive
comments at the point of use, the MCP2518FD package swaps its 1uF bulk
capacitor to a 0603 part to match the current sizing rule, and several
packages add better net-name overrides for exposed and important internal
signals.

Constraint: Repo guidance now prefers explicit local parts and expects readable schematic net names
Constraint: Passive sizing should follow the current MLCC package rule unless a justified exception is needed
Rejected: Keep part instances comment-free | explicit local part names are not readable enough by themselves
Rejected: Leave the MCP2518FD 1uF bulk cap in 0402 | conflicts with the current 1uF-10uF 0603 guidance
Confidence: medium
Scope-risk: moderate
Reversibility: clean
Directive: When instantiating explicit local resistor/capacitor parts, include a short readable comment with the key value/package characteristics unless the name is already obviously human-readable
Tested:  passed for stm32g0b1kbu6_st, mcp2518fdt_e_sl_microchip, tcan3413ddfr_ti, raspberry_pi_hat_socket_zhouri, bq40z50rsmr_r2_4s_3a_ti, tps56637rpar_5v1_5a_ti, tps62933drlr_3v3_ti, bq25756rrvr_4s_2a_ti, tps2121ruxr_20v_4a_ti, and tps25730drefr_20v_3a_ti
Not-tested: Complete elimination of all internal autogenerated net labels in every package; some deep internal nets may still remain tool-driven
Connections:
- net lv renamed GND
- C2 pad 1: hv -> VIN
- C3 pad 1: hv -> VIN
- C4 pad 1: hv -> VIN
- C5 pad 1: power_out-hv -> hv
- C6 pad 1: power_out-hv -> hv
- L1 pad 2: power_out-hv -> hv
- R2 pad 1: power_out-hv -> hv
- U1 pad 2: hv -> VIN
- U1 pad 3: hv -> VIN
Changed lines of the file:
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@@
 	(net 4 "SS")
 	(net 5 "FB")
-	(net 6 "hv")
-	(net 8 "lv")
+	(net 6 "VIN")
+	(net 8 "GND")
 	(net 2 "SW")
-	(net 7 "power_out-hv")
+	(net 7 "hv")
 	(footprint "Texas_Instruments_TPS62933DRLR:SOT-583-8_L2.1-W1.2-P0.50-LS1.6-BR"
 		(layer "F.Cu")
@@
 			(size 0.28 0.68)
 			(layers "F.Cu" "F.Paste" "F.Mask")
-			(net 8 "lv")
+			(net 8 "GND")
 		)
 		(pad "3" smd rect
@@
 			(size 0.28 0.68)
 			(layers "F.Cu" "F.Paste" "F.Mask")
-			(net 6 "hv")
+			(net 6 "VIN")
 		)
 		(pad "2" smd rect
@@
 			(size 0.28 0.68)
 			(layers "F.Cu" "F.Paste" "F.Mask")
-			(net 6 "hv")
+			(net 6 "VIN")
 		)
 		(pad "1" smd rect
@@
 			(size 0.28 0.68)
 			(layers "F.Cu" "F.Paste" "F.Mask")
-			(net 8 "lv")
+			(net 8 "GND")
 		)
 		(embedded_fonts no)
@@
 			(size 0.5 0.54)
 			(layers "F.Cu" "F.Paste" "F.Mask")
-			(net 8 "lv")
+			(net 8 "GND")
 		)
 		(pad "1" smd rect
@@
 			(size 0.5 0.54)
 			(layers "F.Cu" "F.Paste" "F.Mask")
-			(net 6 "hv")
+			(net 6 "VIN")
 		)
 		(embedded_fonts no)
@@
 			(size 0.57 0.54)
 			(layers "F.Cu" "F.Paste" "F.Mask")
-			(net 8 "lv")
+			(net 8 "GND")
 		)
 		(pad "1" smd rect
@@
 			(size 0.57 0.54)
 			(layers "F.Cu" "F.Paste" "F.Mask")
-			(net 7 "power_out-hv")
+			(net 7 "hv")
 		)
 		(embedded_fonts no)
@@
 			(size 1.49 1.73)
 			(layers "F.Cu" "F.Paste" "F.Mask")
-			(net 8 "lv")
+			(net 8 "GND")
 		)
 		(pad "1" smd rect
@@
 			(size 1.49 1.73)
 			(layers "F.Cu" "F.Paste" "F.Mask")
-			(net 6 "hv")
+			(net 6 "VIN")
 		)
 		(embedded_fonts no)
@@
 			(size 1.49 1.73)
 			(layers "F.Cu" "F.Paste" "F.Mask")
-			(net 8 "lv")
+			(net 8 "GND")
 		)
 		(pad "1" smd rect
@@
 			(size 1.49 1.73)
 			(layers "F.Cu" "F.Paste" "F.Mask")
-			(net 6 "hv")
+			(net 6 "VIN")
 		)
 		(embedded_fonts no)
@@
 			(size 1.49 1.73)
 			(layers "F.Cu" "F.Paste" "F.Mask")
-			(net 8 "lv")
+			(net 8 "GND")
 		)
 		(pad "1" smd rect
@@
 			(size 1.49 1.73)
 			(layers "F.Cu" "F.Paste" "F.Mask")
-			(net 7 "power_out-hv")
+			(net 7 "hv")
 		)
 		(embedded_fonts no)
@@
 			(size 1.49 1.73)
 			(layers "F.Cu" "F.Paste" "F.Mask")
-			(net 8 "lv")
+			(net 8 "GND")
 		)
 		(pad "1" smd rect
@@
 			(size 1.49 1.73)
 			(layers "F.Cu" "F.Paste" "F.Mask")
-			(net 7 "power_out-hv")
+			(net 7 "hv")
 		)
 		(embedded_fonts no)
@@
 			(size 2.2 0.8)
 			(layers "F.Cu" "F.Paste" "F.Mask")
-			(net 7 "power_out-hv")
+			(net 7 "hv")
 		)
 		(pad "1" smd rect
@@
 			(size 0.5 0.54)
 			(layers "F.Cu" "F.Paste" "F.Mask")
-			(net 8 "lv")
+			(net 8 "GND")
 		)
 		(pad "1" smd rect

Commit message: Finish removing net-name overrides from reusable packages
This completes the package-level override cleanup by deleting the remaining
`override_net_name` assignments from the library's reusable package modules and
rebuilding their checked-in layouts so generated net metadata matches source.
The package interfaces stay the same; only the forced net naming was removed so
these modules compose cleanly when imported into downstream designs.

Constraint: The library must stay reusable and avoid imposed internal net names leaking into consuming designs
Constraint: Each changed package must still verify with the repo's Atopile workflow after layout regeneration
Rejected: Stop after the battery frontend cleanup | leaves the same composition hazard in other packages
Rejected: Remove override lines without rebuilding layouts | would leave stale generated PCB net names checked into the repo
Confidence: high
Scope-risk: moderate
Reversibility: clean
Directive: Do not reintroduce `override_net_name` in reusable package modules unless a package is intentionally design-specific
Tested: `uv tool run --from atopile==0.15.4 ato --non-interactive build` in each affected package directory (stm32g0b1kbu6_st, mcp2518fdt_e_sl_microchip, tcan3413ddfr_ti, raspberry_pi_hat_socket_zhouri, tps56637rpar_5v1_5a_ti, tps62933drlr_3v3_ti, bq25756rrvr_4s_2a_ti, tps2121ruxr_20v_4a_ti, tps25730drefr_20v_3a_ti)
Not-tested: Downstream consumer projects that may have been depending on the old forced net names in generated layouts
Connections:
- net GND renamed lv
- C2 pad 1: VIN -> hv
- C3 pad 1: VIN -> hv
- C4 pad 1: VIN -> hv
- C5 pad 1: hv -> power_out-hv
- C6 pad 1: hv -> power_out-hv
- L1 pad 2: hv -> power_out-hv
- R2 pad 1: hv -> power_out-hv
- U1 pad 2: VIN -> hv
- U1 pad 3: VIN -> hv
Changed lines of the file:
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@@
 	(net 4 "SS")
 	(net 5 "FB")
-	(net 6 "VIN")
-	(net 8 "GND")
+	(net 6 "hv")
+	(net 8 "lv")
 	(net 2 "SW")
-	(net 7 "hv")
+	(net 7 "power_out-hv")
 	(footprint "Texas_Instruments_TPS62933DRLR:SOT-583-8_L2.1-W1.2-P0.50-LS1.6-BR"
 		(layer "F.Cu")
@@
 			(size 0.28 0.68)
 			(layers "F.Cu" "F.Paste" "F.Mask")
-			(net 8 "GND")
+			(net 8 "lv")
 		)
 		(pad "3" smd rect
@@
 			(size 0.28 0.68)
 			(layers "F.Cu" "F.Paste" "F.Mask")
-			(net 6 "VIN")
+			(net 6 "hv")
 		)
 		(pad "2" smd rect
@@
 			(size 0.28 0.68)
 			(layers "F.Cu" "F.Paste" "F.Mask")
-			(net 6 "VIN")
+			(net 6 "hv")
 		)
 		(pad "1" smd rect
@@
 			(size 0.28 0.68)
 			(layers "F.Cu" "F.Paste" "F.Mask")
-			(net 8 "GND")
+			(net 8 "lv")
 		)
 		(embedded_fonts no)
@@
 			(size 0.5 0.54)
 			(layers "F.Cu" "F.Paste" "F.Mask")
-			(net 8 "GND")
+			(net 8 "lv")
 		)
 		(pad "1" smd rect
@@
 			(size 0.5 0.54)
 			(layers "F.Cu" "F.Paste" "F.Mask")
-			(net 6 "VIN")
+			(net 6 "hv")
 		)
 		(embedded_fonts no)
@@
 			(size 0.57 0.54)
 			(layers "F.Cu" "F.Paste" "F.Mask")
-			(net 8 "GND")
+			(net 8 "lv")
 		)
 		(pad "1" smd rect
@@
 			(size 0.57 0.54)
 			(layers "F.Cu" "F.Paste" "F.Mask")
-			(net 7 "hv")
+			(net 7 "power_out-hv")
 		)
 		(embedded_fonts no)
@@
 			(size 1.49 1.73)
 			(layers "F.Cu" "F.Paste" "F.Mask")
-			(net 8 "GND")
+			(net 8 "lv")
 		)
 		(pad "1" smd rect
@@
 			(size 1.49 1.73)
 			(layers "F.Cu" "F.Paste" "F.Mask")
-			(net 6 "VIN")
+			(net 6 "hv")
 		)
 		(embedded_fonts no)
@@
 			(size 1.49 1.73)
 			(layers "F.Cu" "F.Paste" "F.Mask")
-			(net 8 "GND")
+			(net 8 "lv")
 		)
 		(pad "1" smd rect
@@
 			(size 1.49 1.73)
 			(layers "F.Cu" "F.Paste" "F.Mask")
-			(net 6 "VIN")
+			(net 6 "hv")
 		)
 		(embedded_fonts no)
@@
 			(size 1.49 1.73)
 			(layers "F.Cu" "F.Paste" "F.Mask")
-			(net 8 "GND")
+			(net 8 "lv")
 		)
 		(pad "1" smd rect
@@
 			(size 1.49 1.73)
 			(layers "F.Cu" "F.Paste" "F.Mask")
-			(net 7 "hv")
+			(net 7 "power_out-hv")
 		)
 		(embedded_fonts no)
@@
 			(size 1.49 1.73)
 			(layers "F.Cu" "F.Paste" "F.Mask")
-			(net 8 "GND")
+			(net 8 "lv")
 		)
 		(pad "1" smd rect
@@
 			(size 1.49 1.73)
 			(layers "F.Cu" "F.Paste" "F.Mask")
-			(net 7 "hv")
+			(net 7 "power_out-hv")
 		)
 		(embedded_fonts no)
@@
 			(size 2.2 0.8)
 			(layers "F.Cu" "F.Paste" "F.Mask")
-			(net 7 "hv")
+			(net 7 "power_out-hv")
 		)
 		(pad "1" smd rect
@@
 			(size 0.5 0.54)
 			(layers "F.Cu" "F.Paste" "F.Mask")
-			(net 8 "GND")
+			(net 8 "lv")
 		)
 		(pad "1" smd rect
