File: packages/power/usb_pd/tps25730drefr_20v_3a_ti/layouts/example/example.kicad_pcb (KiCad board)
At the start: 2 copper layers, 9 parts

Commit message: Finish removing net-name overrides from reusable packages
This completes the package-level override cleanup by deleting the remaining
`override_net_name` assignments from the library's reusable package modules and
rebuilding their checked-in layouts so generated net metadata matches source.
The package interfaces stay the same; only the forced net naming was removed so
these modules compose cleanly when imported into downstream designs.

Constraint: The library must stay reusable and avoid imposed internal net names leaking into consuming designs
Constraint: Each changed package must still verify with the repo's Atopile workflow after layout regeneration
Rejected: Stop after the battery frontend cleanup | leaves the same composition hazard in other packages
Rejected: Remove override lines without rebuilding layouts | would leave stale generated PCB net names checked into the repo
Confidence: high
Scope-risk: moderate
Reversibility: clean
Directive: Do not reintroduce `override_net_name` in reusable package modules unless a package is intentionally design-specific
Tested: `uv tool run --from atopile==0.15.4 ato --non-interactive build` in each affected package directory (stm32g0b1kbu6_st, mcp2518fdt_e_sl_microchip, tcan3413ddfr_ti, raspberry_pi_hat_socket_zhouri, tps56637rpar_5v1_5a_ti, tps62933drlr_3v3_ti, bq25756rrvr_4s_2a_ti, tps2121ruxr_20v_4a_ti, tps25730drefr_20v_3a_ti)
Not-tested: Downstream consumer projects that may have been depending on the old forced net names in generated layouts
Connections:
- net 3V3 renamed hv
- net CC1 renamed cc1-1
- net CC2 renamed cc2-1
- net GND renamed lv
- net LDO_1V5 renamed controller-1
- net LDO_3V3 renamed adc_limit_top-1
- net PD_LIMIT_SEL renamed 1
- net SINK_VBUS renamed sink_vbus-hv
- net USB_VBUS renamed usb_vbus-hv
Changed lines of the file:
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@@
 		)
 	)
-	(net 2 "CC1")
-	(net 3 "CC2")
-	(net 4 "LDO_3V3")
+	(net 2 "cc1-1")
+	(net 3 "cc2-1")
+	(net 4 "adc_limit_top-1")
 	(net 5 "DBG_ACC")
 	(net 6 "PLUG_FLIP")
-	(net 7 "GND")
+	(net 7 "lv")
 	(net 8 "nSINK_EN")
-	(net 9 "USB_VBUS")
+	(net 9 "usb_vbus-hv")
 	(net 10 "PLUG_EVENT")
-	(net 11 "3V3")
+	(net 11 "hv")
 	(net 12 "CAP_MIS")
-	(net 13 "PD_LIMIT_SEL")
+	(net 13 "1")
 	(net 14 "SDA")
 	(net 15 "SCL")
-	(net 16 "LDO_1V5")
-	(net 17 "SINK_VBUS")
+	(net 16 "controller-1")
+	(net 17 "sink_vbus-hv")
 	(footprint "TEXAS_INSTRUMENTS_TPS25730DREFR:QFN-38_L6.0-W4.0-P0.40-TL-EP_RJK"
 		(layer "F.Cu")
@@
 			(size 0.6 0.2)
 			(layers "F.Cu" "F.Paste" "F.Mask")
-			(net 4 "LDO_3V3")
+			(net 4 "adc_limit_top-1")
 		)
 		(pad "2" smd rect
@@
 			(size 0.6 0.2)
 			(layers "F.Cu" "F.Paste" "F.Mask")
-			(net 7 "GND")
+			(net 7 "lv")
 		)
 		(pad "3" smd rect
@@
 			(size 0.6 0.2)
 			(layers "F.Cu" "F.Paste" "F.Mask")
-			(net 4 "LDO_3V3")
+			(net 4 "adc_limit_top-1")
 		)
 		(pad "4" smd rect
@@
 			(size 0.6 0.2)
 			(layers "F.Cu" "F.Paste" "F.Mask")
-			(net 16 "LDO_1V5")
+			(net 16 "controller-1")
 		)
 		(pad "5" smd rect
@@
 			(size 0.6 0.2)
 			(layers "F.Cu" "F.Paste" "F.Mask")
-			(net 7 "GND")
+			(net 7 "lv")
 		)
 		(pad "6" smd rect
@@
 			(size 0.2 0.6)
 			(layers "F.Cu" "F.Paste" "F.Mask")
-			(net 13 "PD_LIMIT_SEL")
+			(net 13 "1")
 		)
 		(pad "8" smd rect
@@
 			(size 0.2 0.6)
 			(layers "F.Cu" "F.Paste" "F.Mask")
-			(net 7 "GND")
+			(net 7 "lv")
 		)
 		(pad "12" smd rect
@@
 			(size 0.2 0.6)
 			(layers "F.Cu" "F.Paste" "F.Mask")
-			(net 7 "GND")
+			(net 7 "lv")
 		)
 		(pad "13" smd rect
@@
 			(size 0.2 0.6)
 			(layers "F.Cu" "F.Paste" "F.Mask")
-			(net 7 "GND")
+			(net 7 "lv")
 		)
 		(pad "15" smd rect
@@
 			(size 0.2 0.6)
 			(layers "F.Cu" "F.Paste" "F.Mask")
-			(net 9 "USB_VBUS")
+			(net 9 "usb_vbus-hv")
 		)
 		(pad "16" smd rect
@@
 			(size 0.2 0.6)
 			(layers "F.Cu" "F.Paste" "F.Mask")
-			(net 7 "GND")
+			(net 7 "lv")
 		)
 		(pad "17" smd rect
@@
 			(size 0.2 0.6)
 			(layers "F.Cu" "F.Paste" "F.Mask")
-			(net 7 "GND")
+			(net 7 "lv")
 		)
 		(pad "18" smd rect
@@
 			(size 0.2 0.6)
 			(layers "F.Cu" "F.Paste" "F.Mask")
-			(net 4 "LDO_3V3")
+			(net 4 "adc_limit_top-1")
 		)
 		(pad "19" smd rect
@@
 			(size 0.6 0.22)
 			(layers "F.Cu" "F.Paste" "F.Mask")
-			(net 17 "SINK_VBUS")
+			(net 17 "sink_vbus-hv")
 		)
 		(pad "21" smd rect
@@
 			(size 0.6 0.22)
 			(layers "F.Cu" "F.Paste" "F.Mask")
-			(net 17 "SINK_VBUS")
+			(net 17 "sink_vbus-hv")
 		)
 		(pad "22" smd rect
@@
 			(size 0.6 0.22)
 			(layers "F.Cu" "F.Paste" "F.Mask")
-			(net 17 "SINK_VBUS")
+			(net 17 "sink_vbus-hv")
 		)
 		(pad "23" smd rect
@@
 			(size 0.6 0.22)
 			(layers "F.Cu" "F.Paste" "F.Mask")
-			(net 9 "USB_VBUS")
+			(net 9 "usb_vbus-hv")
 		)
 		(pad "24" smd rect
@@
 			(size 0.6 0.22)
 			(layers "F.Cu" "F.Paste" "F.Mask")
-			(net 9 "USB_VBUS")
+			(net 9 "usb_vbus-hv")
 		)
 		(pad "25" smd rect
@@
 			(size 0.6 0.22)
 			(layers "F.Cu" "F.Paste" "F.Mask")
-			(net 9 "USB_VBUS")
+			(net 9 "usb_vbus-hv")
 		)
 		(pad "26" smd rect
@@
 			(size 0.2 0.6)
 			(layers "F.Cu" "F.Paste" "F.Mask")
-			(net 7 "GND")
+			(net 7 "lv")
 		)
 		(pad "27" smd rect
@@
 			(size 0.2 0.6)
 			(layers "F.Cu" "F.Paste" "F.Mask")
-			(net 7 "GND")
+			(net 7 "lv")
 		)
 		(pad "28" smd rect
@@
 			(size 0.2 0.6)
 			(layers "F.Cu" "F.Paste" "F.Mask")
-			(net 2 "CC1")
+			(net 2 "cc1-1")
 		)
 		(pad "29" smd rect
@@
 			(size 0.2 0.6)
 			(layers "F.Cu" "F.Paste" "F.Mask")
-			(net 3 "CC2")
+			(net 3 "cc2-1")
 		)
 		(pad "30" smd rect
@@
 			(size 0.2 0.6)
 			(layers "F.Cu" "F.Paste" "F.Mask")
-			(net 9 "USB_VBUS")
+			(net 9 "usb_vbus-hv")
 		)
 		(pad "31" smd rect
@@
 			(size 0.2 0.6)
 			(layers "F.Cu" "F.Paste" "F.Mask")
-			(net 7 "GND")
+			(net 7 "lv")
 		)
 		(pad "32" smd rect
@@
 			(size 0.2 0.6)
 			(layers "F.Cu" "F.Paste" "F.Mask")
-			(net 9 "USB_VBUS")
+			(net 9 "usb_vbus-hv")
 		)
 		(pad "33" smd rect
@@
 			(size 0.2 0.6)
 			(layers "F.Cu" "F.Paste" "F.Mask")
-			(net 9 "USB_VBUS")
+			(net 9 "usb_vbus-hv")
 		)
 		(pad "34" smd rect
@@
 			(size 0.2 0.6)
 			(layers "F.Cu" "F.Paste" "F.Mask")
-			(net 7 "GND")
+			(net 7 "lv")
 		)
 		(pad "35" smd rect
@@
 			(size 0.2 0.6)
 			(layers "F.Cu" "F.Paste" "F.Mask")
-			(net 7 "GND")
+			(net 7 "lv")
 		)
 		(pad "36" smd rect
@@
 			(size 0.2 0.6)
 			(layers "F.Cu" "F.Paste" "F.Mask")
-			(net 7 "GND")
+			(net 7 "lv")
 		)
 		(pad "37" smd rect
@@
 			(size 0.2 0.6)
 			(layers "F.Cu" "F.Paste" "F.Mask")
-			(net 11 "3V3")
+			(net 11 "hv")
 		)
 		(pad "39" smd rect
@@
 			(size 2.65 2.65)
 			(layers "F.Cu" "F.Paste" "F.Mask")
-			(net 7 "GND")
+			(net 7 "lv")
 		)
 		(pad "35" smd custom
@@
 			(size 0.01 0.01)
 			(layers "F.Cu" "F.Paste" "F.Mask")
-			(net 7 "GND")
+			(net 7 "lv")
 			(primitives
 				(gr_poly
@@
 			(size 0.01 0.01)
 			(layers "F.Cu" "F.Paste" "F.Mask")
-			(net 9 "USB_VBUS")
+			(net 9 "usb_vbus-hv")
 			(primitives
 				(gr_poly
@@
 			(size 0.01 0.01)
 			(layers "F.Cu" "F.Paste" "F.Mask")
-			(net 9 "USB_VBUS")
+			(net 9 "usb_vbus-hv")
 			(primitives
 				(gr_poly
@@
 			(size 0.01 0.01)
 			(layers "F.Cu" "F.Paste" "F.Mask")
-			(net 17 "SINK_VBUS")
+			(net 17 "sink_vbus-hv")
 			(primitives
 				(gr_poly
@@
 			(size 1.53 2.65)
 			(layers "F.Cu" "F.Paste" "F.Mask")
-			(net 9 "USB_VBUS")
+			(net 9 "usb_vbus-hv")
 		)
 		(embedded_fonts no)
@@
 			(size 0.57 0.54)
 			(layers "F.Cu" "F.Paste" "F.Mask")
-			(net 7 "GND")
+			(net 7 "lv")
 		)
 		(pad "1" smd rect
@@
 			(size 0.57 0.54)
 			(layers "F.Cu" "F.Paste" "F.Mask")
-			(net 13 "PD_LIMIT_SEL")
+			(net 13 "1")
 		)
 		(embedded_fonts no)
@@
 			(size 0.57 0.54)
 			(layers "F.Cu" "F.Paste" "F.Mask")
-			(net 13 "PD_LIMIT_SEL")
+			(net 13 "1")
 		)
 		(pad "1" smd rect
@@
 			(size 0.57 0.54)
 			(layers "F.Cu" "F.Paste" "F.Mask")
-			(net 4 "LDO_3V3")
+			(net 4 "adc_limit_top-1")
 		)
 		(embedded_fonts no)
@@
 			(size 0.5 0.54)
 			(layers "F.Cu" "F.Paste" "F.Mask")
-			(net 7 "GND")
+			(net 7 "lv")
 		)
 		(pad "1" smd rect
@@
 			(size 0.5 0.54)
 			(layers "F.Cu" "F.Paste" "F.Mask")
-			(net 2 "CC1")
+			(net 2 "cc1-1")
 		)
 		(embedded_fonts no)
@@
 			(size 0.5 0.54)
 			(layers "F.Cu" "F.Paste" "F.Mask")
-			(net 7 "GND")
+			(net 7 "lv")
 		)
 		(pad "1" smd rect
@@
 			(size 0.5 0.54)
 			(layers "F.Cu" "F.Paste" "F.Mask")
-			(net 3 "CC2")
+			(net 3 "cc2-1")
 		)
 		(embedded_fonts no)
@@
 			(size 0.5 0.54)
 			(layers "F.Cu" "F.Paste" "F.Mask")
-			(net 7 "GND")
+			(net 7 "lv")
 		)
 		(pad "1" smd rect
@@
 			(size 0.5 0.54)
 			(layers "F.Cu" "F.Paste" "F.Mask")
-			(net 16 "LDO_1V5")
+			(net 16 "controller-1")
 		)
 		(embedded_fonts no)
@@
 			(size 0.8 0.9)
 			(layers "F.Cu" "F.Paste" "F.Mask")
-			(net 7 "GND")
+			(net 7 "lv")
 		)
 		(pad "1" smd rect
@@
 			(size 0.8 0.9)
 			(layers "F.Cu" "F.Paste" "F.Mask")
-			(net 4 "LDO_3V3")
+			(net 4 "adc_limit_top-1")
 		)
 		(embedded_fonts no)
@@
 			(size 0.8 0.9)
 			(layers "F.Cu" "F.Paste" "F.Mask")
-			(net 7 "GND")
+			(net 7 "lv")
 		)
 		(pad "1" smd rect
@@
 			(size 0.8 0.9)
 			(layers "F.Cu" "F.Paste" "F.Mask")
-			(net 11 "3V3")
+			(net 11 "hv")
 		)
 		(embedded_fonts no)
@@
 			(size 0.8 0.9)
 			(layers "F.Cu" "F.Paste" "F.Mask")
-			(net 7 "GND")
+			(net 7 "lv")
 		)
 		(pad "1" smd rect
@@
 			(size 0.8 0.9)
 			(layers "F.Cu" "F.Paste" "F.Mask")
-			(net 9 "USB_VBUS")
+			(net 9 "usb_vbus-hv")
 		)
 		(embedded_fonts no)
