File: packages/power/buck/tps56637rpar_5v1_5a_ti/layouts/default/default.kicad_pcb (KiCad board)
At the start: 2 copper layers, 10 parts

Commit message: Make package builds deterministic by wiring explicit local parts
The remaining packages now reference package-local concrete passives,
inductors, and other small parts directly instead of relying on generic
part-picker resolution. This aligns the source with the local
assets and removes the flaky live EasyEDA lookup path that was blocking
verification.

Constraint: Builds must not depend on unstable live part-picking when local package assets already exist
Constraint: Package-local parts remain the ownership boundary; no shared global part store was introduced
Rejected: Keep generic passives as the default style | repeated verification failures from upstream EasyEDA API instability
Rejected: Add ad hoc offline hacks around ato part-picking | weaker than making the package source deterministic
Confidence: high
Scope-risk: moderate
Reversibility: clean
Directive: For packages that already own generated local parts, instantiate those part modules directly and avoid generic passive declarations unless there is a strong reason not to
Tested:  passed for stm32g0b1kbu6_st, mcp2518fdt_e_sl_microchip, tcan3413ddfr_ti, raspberry_pi_hat_socket_zhouri, bq40z50rsmr_r2_4s_3a_ti, tps56637rpar_5v1_5a_ti, tps62933drlr_3v3_ti, bq25756rrvr_4s_2a_ti, tps2121ruxr_20v_4a_ti, and tps25730drefr_20v_3a_ti
Not-tested: Cross-package downstream integration beyond each package's default/example build
Parts:
- C1, C2, C3, C4, C5, C6: value 0F -> (none)
- L1: value L 0H -> (none)
- R1: value 10000Ω -> (none)
- R2: value 75000Ω -> (none)
Connections:
- net FB renamed 2
- net output_bulk_b-power-hv renamed power_out-hv
- C1 pad 1: hv -> BOOT
- C1 pad 2: lv -> SW
- C2 pad 1: input_bypass-power-hv -> hv
- C2 pad 2: output_bulk_b-power-lv -> lv
- C3 pad 1: input_bypass-power-hv -> hv
- C3 pad 2: output_bulk_b-power-lv -> lv
- C4 pad 1: input_bypass-power-hv -> hv
- C4 pad 2: output_bulk_b-power-lv -> lv
- C5 pad 2: output_bulk_b-power-lv -> lv
- C6 pad 2: output_bulk_b-power-lv -> lv
- L1 pad 1: lv -> SW
- R1 pad 2: output_bulk_b-power-lv -> lv
- U1 pad 3: output_bulk_b-power-lv -> lv
- U1 pad 6: lv -> SW
- U1 pad 7: hv -> BOOT
- U1 pad 8: input_bypass-power-hv -> hv
- U1 pad 9: output_bulk_b-power-lv -> lv
Changed lines of the file:
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@@
 		)
 	)
-	(net 1 "lv")
+	(net 1 "SW")
 	(net 2 "EN")
 	(net 3 "MODE")
-	(net 4 "FB")
+	(net 4 "2")
 	(net 5 "PG")
-	(net 6 "hv")
-	(net 7 "input_bypass-power-hv")
-	(net 8 "output_bulk_b-power-lv")
-	(net 9 "output_bulk_b-power-hv")
+	(net 6 "BOOT")
+	(net 7 "hv")
+	(net 8 "lv")
+	(net 9 "power_out-hv")
 	(footprint "Texas_Instruments_TPS56637RPAR:VQFN-HR-10_L3.0-W3.0_RPA"
 		(layer "F.Cu")
@@
 			(locked no)
 		)
-		(fp_text user "%R"
-			(at 0 0)
-			(layer "F.Fab")
-			(effects
-				(font
-					(size 1 1)
-					(thickness 0.15)
-				)
-			)
-		)
 		(pad "8" smd rect
 			(at 0.99 -0.65 0)
 			(size 0.4 2.1)
 			(layers "F.Cu" "F.Paste" "F.Mask")
-			(net 7 "input_bypass-power-hv")
+			(net 7 "hv")
 		)
 		(pad "10" smd rect
@@
 			(size 0.4 2.1)
 			(layers "F.Cu" "F.Paste" "F.Mask")
-			(net 8 "output_bulk_b-power-lv")
+			(net 8 "lv")
 		)
 		(pad "5" smd rect
@@
 			(size 0.25 1.7)
 			(layers "F.Cu" "F.Paste" "F.Mask")
-			(net 1 "lv")
+			(net 1 "SW")
 		)
 		(pad "7" smd rect
@@
 			(size 0.6 0.25)
 			(layers "F.Cu" "F.Paste" "F.Mask")
-			(net 6 "hv")
+			(net 6 "BOOT")
 		)
 		(pad "8" smd rect
@@
 			(size 0.8 0.25)
 			(layers "F.Cu" "F.Paste" "F.Mask")
-			(net 7 "input_bypass-power-hv")
+			(net 7 "hv")
 		)
 		(pad "8" smd rect
@@
 			(size 0.8 0.25)
 			(layers "F.Cu" "F.Paste" "F.Mask")
-			(net 7 "input_bypass-power-hv")
+			(net 7 "hv")
 		)
 		(pad "8" smd rect
@@
 			(size 0.8 0.25)
 			(layers "F.Cu" "F.Paste" "F.Mask")
-			(net 7 "input_bypass-power-hv")
+			(net 7 "hv")
 		)
 		(pad "4" smd rect
@@
 			(size 0.6 0.25)
 			(layers "F.Cu" "F.Paste" "F.Mask")
-			(net 8 "output_bulk_b-power-lv")
+			(net 8 "lv")
 		)
 		(pad "2" smd rect
@@
 			(size 0.6 0.25)
 			(layers "F.Cu" "F.Paste" "F.Mask")
-			(net 4 "FB")
+			(net 4 "2")
 		)
 		(pad "1" smd rect
@@
 			)
 		)
-		(property "Value" "0F"
+		(property "Value" ""
 			(at 0 4)
 			(layer "F.Fab")
@@
 			(locked no)
 		)
-		(fp_text user "%R"
-			(at 0 0)
-			(layer "F.Fab")
-			(effects
-				(font
-					(size 1 1)
-					(thickness 0.15)
-				)
-			)
-		)
 		(pad "2" smd rect
 			(at 0.42 0 0)
 			(size 0.5 0.54)
 			(layers "F.Cu" "F.Paste" "F.Mask")
-			(net 1 "lv")
+			(net 1 "SW")
 		)
 		(pad "1" smd rect
@@
 			(size 0.5 0.54)
 			(layers "F.Cu" "F.Paste" "F.Mask")
-			(net 6 "hv")
+			(net 6 "BOOT")
 		)
 		(embedded_fonts no)
@@
 			)
 		)
-		(property "Value" "0F"
+		(property "Value" ""
 			(at 0 4)
 			(layer "F.Fab")
@@
 			(locked no)
 		)
-		(fp_text user "%R"
-			(at 0 0)
-			(layer "F.Fab")
-			(effects
-				(font
-					(size 1 1)
-					(thickness 0.15)
-				)
-			)
-		)
 		(pad "2" smd rect
 			(at 0.42 0 0)
 			(size 0.5 0.54)
 			(layers "F.Cu" "F.Paste" "F.Mask")
-			(net 8 "output_bulk_b-power-lv")
+			(net 8 "lv")
 		)
 		(pad "1" smd rect
@@
 			(size 0.5 0.54)
 			(layers "F.Cu" "F.Paste" "F.Mask")
-			(net 7 "input_bypass-power-hv")
+			(net 7 "hv")
 		)
 		(embedded_fonts no)
@@
 			)
 		)
-		(property "Value" "10000Ω"
+		(property "Value" ""
 			(at 0 4)
 			(layer "F.Fab")
@@
 			(hide yes)
 		)
-		(property "Datasheet" "https://www.lcsc.com/datasheet/lcsc_datasheet_1811141608_YAGEO-RC0402FR-0710KL_C60490.pdf"
+		(property "Datasheet" "https://www.lcsc.com/datasheet/lcsc_datasheet_2304140030_YAGEO-RC0402FR-0710KL_C60490.pdf"
 			(at 0 0 0)
 			(layer "User.9")
@@
 			(locked no)
 		)
-		(fp_text user "%R"
-			(at 0 0)
-			(layer "F.Fab")
-			(effects
-				(font
-					(size 1 1)
-					(thickness 0.15)
-				)
-			)
-		)
 		(pad "2" smd rect
 			(at 0.43 0 0)
 			(size 0.57 0.54)
 			(layers "F.Cu" "F.Paste" "F.Mask")
-			(net 8 "output_bulk_b-power-lv")
+			(net 8 "lv")
 		)
 		(pad "1" smd rect
@@
 			(size 0.57 0.54)
 			(layers "F.Cu" "F.Paste" "F.Mask")
-			(net 4 "FB")
+			(net 4 "2")
 		)
 		(embedded_fonts no)
@@
 			)
 		)
-		(property "Value" "75000Ω"
+		(property "Value" ""
 			(at 0 4)
 			(layer "F.Fab")
@@
 			(hide yes)
 		)
-		(property "Datasheet" "https://www.lcsc.com/datasheet/lcsc_datasheet_1811141608_YAGEO-RC0402FR-0775KL_C137935.pdf"
+		(property "Datasheet" "https://www.lcsc.com/datasheet/lcsc_datasheet_2304140030_YAGEO-RC0402FR-0775KL_C137935.pdf"
 			(at 0 0 0)
 			(layer "User.9")
@@
 			(locked no)
 		)
-		(fp_text user "%R"
-			(at 0 0)
-			(layer "F.Fab")
-			(effects
-				(font
-					(size 1 1)
-					(thickness 0.15)
-				)
-			)
-		)
 		(pad "2" smd rect
 			(at 0.43 0 0)
 			(size 0.57 0.54)
 			(layers "F.Cu" "F.Paste" "F.Mask")
-			(net 4 "FB")
+			(net 4 "2")
 		)
 		(pad "1" smd rect
@@
 			(size 0.57 0.54)
 			(layers "F.Cu" "F.Paste" "F.Mask")
-			(net 9 "output_bulk_b-power-hv")
+			(net 9 "power_out-hv")
 		)
 		(embedded_fonts no)
@@
 			)
 		)
-		(property "Value" "0F"
+		(property "Value" ""
 			(at 0 4)
 			(layer "F.Fab")
@@
 			(locked no)
 		)
-		(fp_text user "%R"
-			(at 0 0)
-			(layer "F.Fab")
-			(effects
-				(font
-					(size 1 1)
-					(thickness 0.15)
-				)
-			)
-		)
 		(pad "2" smd rect
 			(at 1.59 0 0)
 			(size 1.49 1.73)
 			(layers "F.Cu" "F.Paste" "F.Mask")
-			(net 8 "output_bulk_b-power-lv")
+			(net 8 "lv")
 		)
 		(pad "1" smd rect
@@
 			(size 1.49 1.73)
 			(layers "F.Cu" "F.Paste" "F.Mask")
-			(net 7 "input_bypass-power-hv")
+			(net 7 "hv")
 		)
 		(embedded_fonts no)
@@
 			)
 		)
-		(property "Value" "0F"
+		(property "Value" ""
 			(at 0 4)
 			(layer "F.Fab")
@@
 			(locked no)
 		)
-		(fp_text user "%R"
-			(at 0 0)
-			(layer "F.Fab")
-			(effects
-				(font
-					(size 1 1)
-					(thickness 0.15)
-				)
-			)
-		)
 		(pad "2" smd rect
 			(at 1.59 0 0)
 			(size 1.49 1.73)
 			(layers "F.Cu" "F.Paste" "F.Mask")
-			(net 8 "output_bulk_b-power-lv")
+			(net 8 "lv")
 		)
 		(pad "1" smd rect
@@
 			(size 1.49 1.73)
 			(layers "F.Cu" "F.Paste" "F.Mask")
-			(net 7 "input_bypass-power-hv")
+			(net 7 "hv")
 		)
 		(embedded_fonts no)
@@
 			)
 		)
-		(property "Value" "0F"
+		(property "Value" ""
 			(at 0 4)
 			(layer "F.Fab")
@@
 			(locked no)
 		)
-		(fp_text user "%R"
-			(at 0 0)
-			(layer "F.Fab")
-			(effects
-				(font
-					(size 1 1)
-					(thickness 0.15)
-				)
-			)
-		)
 		(pad "2" smd rect
 			(at 1.59 0 0)
 			(size 1.49 1.73)
 			(layers "F.Cu" "F.Paste" "F.Mask")
-			(net 8 "output_bulk_b-power-lv")
+			(net 8 "lv")
 		)
 		(pad "1" smd rect
@@
 			(size 1.49 1.73)
 			(layers "F.Cu" "F.Paste" "F.Mask")
-			(net 9 "output_bulk_b-power-hv")
+			(net 9 "power_out-hv")
 		)
 		(embedded_fonts no)
@@
 			)
 		)
-		(property "Value" "0F"
+		(property "Value" ""
 			(at 0 4)
 			(layer "F.Fab")
@@
 			(locked no)
 		)
-		(fp_text user "%R"
-			(at 0 0)
-			(layer "F.Fab")
-			(effects
-				(font
-					(size 1 1)
-					(thickness 0.15)
-				)
-			)
-		)
 		(pad "2" smd rect
 			(at 1.59 0 0)
 			(size 1.49 1.73)
 			(layers "F.Cu" "F.Paste" "F.Mask")
-			(net 8 "output_bulk_b-power-lv")
+			(net 8 "lv")
 		)
 		(pad "1" smd rect
@@
 			(size 1.49 1.73)
 			(layers "F.Cu" "F.Paste" "F.Mask")
-			(net 9 "output_bulk_b-power-hv")
+			(net 9 "power_out-hv")
 		)
 		(embedded_fonts no)
@@
 			)
 		)
-		(property "Value" "L 0H"
+		(property "Value" ""
 			(at 0 4)
 			(layer "F.Fab")
@@
 			(hide yes)
 		)
-		(property "Manufacturer" "cjiang(Changjiang Microelectronics Tech)"
+		(property "Manufacturer" "cjiang"
 			(at 0 0 0)
 			(layer "User.9")
@@
 			(locked no)
 		)
-		(fp_text user "%R"
-			(at 0 0)
-			(layer "F.Fab")
-			(effects
-				(font
-					(size 1 1)
-					(thickness 0.15)
-				)
-			)
-		)
 		(pad "1" smd rect
 			(at -3 0 0)
 			(size 2.4 3.2)
 			(layers "F.Cu" "F.Paste" "F.Mask")
-			(net 1 "lv")
+			(net 1 "SW")
 		)
 		(pad "2" smd rect
@@
 			(size 2.4 3.2)
 			(layers "F.Cu" "F.Paste" "F.Mask")
-			(net 9 "output_bulk_b-power-hv")
+			(net 9 "power_out-hv")
 		)
 		(embedded_fonts no)

Commit message: Make package schematics more readable and align passive choices with repo guidance
This pass improves the human-facing quality of the package library.
Explicit local capacitor/resistor parts now carry short descriptive
comments at the point of use, the MCP2518FD package swaps its 1uF bulk
capacitor to a 0603 part to match the current sizing rule, and several
packages add better net-name overrides for exposed and important internal
signals.

Constraint: Repo guidance now prefers explicit local parts and expects readable schematic net names
Constraint: Passive sizing should follow the current MLCC package rule unless a justified exception is needed
Rejected: Keep part instances comment-free | explicit local part names are not readable enough by themselves
Rejected: Leave the MCP2518FD 1uF bulk cap in 0402 | conflicts with the current 1uF-10uF 0603 guidance
Confidence: medium
Scope-risk: moderate
Reversibility: clean
Directive: When instantiating explicit local resistor/capacitor parts, include a short readable comment with the key value/package characteristics unless the name is already obviously human-readable
Tested:  passed for stm32g0b1kbu6_st, mcp2518fdt_e_sl_microchip, tcan3413ddfr_ti, raspberry_pi_hat_socket_zhouri, bq40z50rsmr_r2_4s_3a_ti, tps56637rpar_5v1_5a_ti, tps62933drlr_3v3_ti, bq25756rrvr_4s_2a_ti, tps2121ruxr_20v_4a_ti, and tps25730drefr_20v_3a_ti
Not-tested: Complete elimination of all internal autogenerated net labels in every package; some deep internal nets may still remain tool-driven
Connections:
- net 2 renamed FB
- net lv renamed GND
- C2 pad 1: hv -> VIN
- C3 pad 1: hv -> VIN
- C4 pad 1: hv -> VIN
- C5 pad 1: power_out-hv -> hv
- C6 pad 1: power_out-hv -> hv
- L1 pad 2: power_out-hv -> hv
- R2 pad 1: power_out-hv -> hv
- U1 pad 8: hv -> VIN
Changed lines of the file:
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@@
 	(net 2 "EN")
 	(net 3 "MODE")
-	(net 4 "2")
+	(net 4 "FB")
 	(net 5 "PG")
 	(net 6 "BOOT")
-	(net 7 "hv")
-	(net 8 "lv")
-	(net 9 "power_out-hv")
+	(net 7 "VIN")
+	(net 8 "GND")
+	(net 9 "hv")
 	(footprint "Texas_Instruments_TPS56637RPAR:VQFN-HR-10_L3.0-W3.0_RPA"
 		(layer "F.Cu")
@@
 			(size 0.4 2.1)
 			(layers "F.Cu" "F.Paste" "F.Mask")
-			(net 7 "hv")
+			(net 7 "VIN")
 		)
 		(pad "10" smd rect
@@
 			(size 0.4 2.1)
 			(layers "F.Cu" "F.Paste" "F.Mask")
-			(net 8 "lv")
+			(net 8 "GND")
 		)
 		(pad "5" smd rect
@@
 			(size 0.8 0.25)
 			(layers "F.Cu" "F.Paste" "F.Mask")
-			(net 7 "hv")
+			(net 7 "VIN")
 		)
 		(pad "8" smd rect
@@
 			(size 0.8 0.25)
 			(layers "F.Cu" "F.Paste" "F.Mask")
-			(net 7 "hv")
+			(net 7 "VIN")
 		)
 		(pad "8" smd rect
@@
 			(size 0.8 0.25)
 			(layers "F.Cu" "F.Paste" "F.Mask")
-			(net 7 "hv")
+			(net 7 "VIN")
 		)
 		(pad "4" smd rect
@@
 			(size 0.6 0.25)
 			(layers "F.Cu" "F.Paste" "F.Mask")
-			(net 8 "lv")
+			(net 8 "GND")
 		)
 		(pad "2" smd rect
@@
 			(size 0.6 0.25)
 			(layers "F.Cu" "F.Paste" "F.Mask")
-			(net 4 "2")
+			(net 4 "FB")
 		)
 		(pad "1" smd rect
@@
 			(size 0.5 0.54)
 			(layers "F.Cu" "F.Paste" "F.Mask")
-			(net 8 "lv")
+			(net 8 "GND")
 		)
 		(pad "1" smd rect
@@
 			(size 0.5 0.54)
 			(layers "F.Cu" "F.Paste" "F.Mask")
-			(net 7 "hv")
+			(net 7 "VIN")
 		)
 		(embedded_fonts no)
@@
 			(size 0.57 0.54)
 			(layers "F.Cu" "F.Paste" "F.Mask")
-			(net 8 "lv")
+			(net 8 "GND")
 		)
 		(pad "1" smd rect
@@
 			(size 0.57 0.54)
 			(layers "F.Cu" "F.Paste" "F.Mask")
-			(net 4 "2")
+			(net 4 "FB")
 		)
 		(embedded_fonts no)
@@
 			(size 0.57 0.54)
 			(layers "F.Cu" "F.Paste" "F.Mask")
-			(net 4 "2")
+			(net 4 "FB")
 		)
 		(pad "1" smd rect
@@
 			(size 0.57 0.54)
 			(layers "F.Cu" "F.Paste" "F.Mask")
-			(net 9 "power_out-hv")
+			(net 9 "hv")
 		)
 		(embedded_fonts no)
@@
 			(size 1.49 1.73)
 			(layers "F.Cu" "F.Paste" "F.Mask")
-			(net 8 "lv")
+			(net 8 "GND")
 		)
 		(pad "1" smd rect
@@
 			(size 1.49 1.73)
 			(layers "F.Cu" "F.Paste" "F.Mask")
-			(net 7 "hv")
+			(net 7 "VIN")
 		)
 		(embedded_fonts no)
@@
 			(size 1.49 1.73)
 			(layers "F.Cu" "F.Paste" "F.Mask")
-			(net 8 "lv")
+			(net 8 "GND")
 		)
 		(pad "1" smd rect
@@
 			(size 1.49 1.73)
 			(layers "F.Cu" "F.Paste" "F.Mask")
-			(net 7 "hv")
+			(net 7 "VIN")
 		)
 		(embedded_fonts no)
@@
 			(size 1.49 1.73)
 			(layers "F.Cu" "F.Paste" "F.Mask")
-			(net 8 "lv")
+			(net 8 "GND")
 		)
 		(pad "1" smd rect
@@
 			(size 1.49 1.73)
 			(layers "F.Cu" "F.Paste" "F.Mask")
-			(net 9 "power_out-hv")
+			(net 9 "hv")
 		)
 		(embedded_fonts no)
@@
 			(size 1.49 1.73)
 			(layers "F.Cu" "F.Paste" "F.Mask")
-			(net 8 "lv")
+			(net 8 "GND")
 		)
 		(pad "1" smd rect
@@
 			(size 1.49 1.73)
 			(layers "F.Cu" "F.Paste" "F.Mask")
-			(net 9 "power_out-hv")
+			(net 9 "hv")
 		)
 		(embedded_fonts no)
@@
 			(size 2.4 3.2)
 			(layers "F.Cu" "F.Paste" "F.Mask")
-			(net 9 "power_out-hv")
+			(net 9 "hv")
 		)
 		(embedded_fonts no)

Commit message: Finish removing net-name overrides from reusable packages
This completes the package-level override cleanup by deleting the remaining
`override_net_name` assignments from the library's reusable package modules and
rebuilding their checked-in layouts so generated net metadata matches source.
The package interfaces stay the same; only the forced net naming was removed so
these modules compose cleanly when imported into downstream designs.

Constraint: The library must stay reusable and avoid imposed internal net names leaking into consuming designs
Constraint: Each changed package must still verify with the repo's Atopile workflow after layout regeneration
Rejected: Stop after the battery frontend cleanup | leaves the same composition hazard in other packages
Rejected: Remove override lines without rebuilding layouts | would leave stale generated PCB net names checked into the repo
Confidence: high
Scope-risk: moderate
Reversibility: clean
Directive: Do not reintroduce `override_net_name` in reusable package modules unless a package is intentionally design-specific
Tested: `uv tool run --from atopile==0.15.4 ato --non-interactive build` in each affected package directory (stm32g0b1kbu6_st, mcp2518fdt_e_sl_microchip, tcan3413ddfr_ti, raspberry_pi_hat_socket_zhouri, tps56637rpar_5v1_5a_ti, tps62933drlr_3v3_ti, bq25756rrvr_4s_2a_ti, tps2121ruxr_20v_4a_ti, tps25730drefr_20v_3a_ti)
Not-tested: Downstream consumer projects that may have been depending on the old forced net names in generated layouts
Connections:
- net FB renamed 2
- net GND renamed lv
- C2 pad 1: VIN -> hv
- C3 pad 1: VIN -> hv
- C4 pad 1: VIN -> hv
- C5 pad 1: hv -> power_out-hv
- C6 pad 1: hv -> power_out-hv
- L1 pad 2: hv -> power_out-hv
- R2 pad 1: hv -> power_out-hv
- U1 pad 8: VIN -> hv
Changed lines of the file:
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@@
 	(net 2 "EN")
 	(net 3 "MODE")
-	(net 4 "FB")
+	(net 4 "2")
 	(net 5 "PG")
 	(net 6 "BOOT")
-	(net 7 "VIN")
-	(net 8 "GND")
-	(net 9 "hv")
+	(net 7 "hv")
+	(net 8 "lv")
+	(net 9 "power_out-hv")
 	(footprint "Texas_Instruments_TPS56637RPAR:VQFN-HR-10_L3.0-W3.0_RPA"
 		(layer "F.Cu")
@@
 			(size 0.4 2.1)
 			(layers "F.Cu" "F.Paste" "F.Mask")
-			(net 7 "VIN")
+			(net 7 "hv")
 		)
 		(pad "10" smd rect
@@
 			(size 0.4 2.1)
 			(layers "F.Cu" "F.Paste" "F.Mask")
-			(net 8 "GND")
+			(net 8 "lv")
 		)
 		(pad "5" smd rect
@@
 			(size 0.8 0.25)
 			(layers "F.Cu" "F.Paste" "F.Mask")
-			(net 7 "VIN")
+			(net 7 "hv")
 		)
 		(pad "8" smd rect
@@
 			(size 0.8 0.25)
 			(layers "F.Cu" "F.Paste" "F.Mask")
-			(net 7 "VIN")
+			(net 7 "hv")
 		)
 		(pad "8" smd rect
@@
 			(size 0.8 0.25)
 			(layers "F.Cu" "F.Paste" "F.Mask")
-			(net 7 "VIN")
+			(net 7 "hv")
 		)
 		(pad "4" smd rect
@@
 			(size 0.6 0.25)
 			(layers "F.Cu" "F.Paste" "F.Mask")
-			(net 8 "GND")
+			(net 8 "lv")
 		)
 		(pad "2" smd rect
@@
 			(size 0.6 0.25)
 			(layers "F.Cu" "F.Paste" "F.Mask")
-			(net 4 "FB")
+			(net 4 "2")
 		)
 		(pad "1" smd rect
@@
 			(size 0.5 0.54)
 			(layers "F.Cu" "F.Paste" "F.Mask")
-			(net 8 "GND")
+			(net 8 "lv")
 		)
 		(pad "1" smd rect
@@
 			(size 0.5 0.54)
 			(layers "F.Cu" "F.Paste" "F.Mask")
-			(net 7 "VIN")
+			(net 7 "hv")
 		)
 		(embedded_fonts no)
@@
 			(size 0.57 0.54)
 			(layers "F.Cu" "F.Paste" "F.Mask")
-			(net 8 "GND")
+			(net 8 "lv")
 		)
 		(pad "1" smd rect
@@
 			(size 0.57 0.54)
 			(layers "F.Cu" "F.Paste" "F.Mask")
-			(net 4 "FB")
+			(net 4 "2")
 		)
 		(embedded_fonts no)
@@
 			(size 0.57 0.54)
 			(layers "F.Cu" "F.Paste" "F.Mask")
-			(net 4 "FB")
+			(net 4 "2")
 		)
 		(pad "1" smd rect
@@
 			(size 0.57 0.54)
 			(layers "F.Cu" "F.Paste" "F.Mask")
-			(net 9 "hv")
+			(net 9 "power_out-hv")
 		)
 		(embedded_fonts no)
@@
 			(size 1.49 1.73)
 			(layers "F.Cu" "F.Paste" "F.Mask")
-			(net 8 "GND")
+			(net 8 "lv")
 		)
 		(pad "1" smd rect
@@
 			(size 1.49 1.73)
 			(layers "F.Cu" "F.Paste" "F.Mask")
-			(net 7 "VIN")
+			(net 7 "hv")
 		)
 		(embedded_fonts no)
@@
 			(size 1.49 1.73)
 			(layers "F.Cu" "F.Paste" "F.Mask")
-			(net 8 "GND")
+			(net 8 "lv")
 		)
 		(pad "1" smd rect
@@
 			(size 1.49 1.73)
 			(layers "F.Cu" "F.Paste" "F.Mask")
-			(net 7 "VIN")
+			(net 7 "hv")
 		)
 		(embedded_fonts no)
@@
 			(size 1.49 1.73)
 			(layers "F.Cu" "F.Paste" "F.Mask")
-			(net 8 "GND")
+			(net 8 "lv")
 		)
 		(pad "1" smd rect
@@
 			(size 1.49 1.73)
 			(layers "F.Cu" "F.Paste" "F.Mask")
-			(net 9 "hv")
+			(net 9 "power_out-hv")
 		)
 		(embedded_fonts no)
@@
 			(size 1.49 1.73)
 			(layers "F.Cu" "F.Paste" "F.Mask")
-			(net 8 "GND")
+			(net 8 "lv")
 		)
 		(pad "1" smd rect
@@
 			(size 1.49 1.73)
 			(layers "F.Cu" "F.Paste" "F.Mask")
-			(net 9 "hv")
+			(net 9 "power_out-hv")
 		)
 		(embedded_fonts no)
@@
 			(size 2.4 3.2)
 			(layers "F.Cu" "F.Paste" "F.Mask")
-			(net 9 "hv")
+			(net 9 "power_out-hv")
 		)
 		(embedded_fonts no)
