File: packages/power/charger/bq25756rrvr_4s_2a_ti/layouts/default/default.kicad_pcb (KiCad board)
At the start: 2 copper layers, 29 parts

Commit message: Make package builds deterministic by wiring explicit local parts
The remaining packages now reference package-local concrete passives,
inductors, and other small parts directly instead of relying on generic
part-picker resolution. This aligns the source with the local
assets and removes the flaky live EasyEDA lookup path that was blocking
verification.

Constraint: Builds must not depend on unstable live part-picking when local package assets already exist
Constraint: Package-local parts remain the ownership boundary; no shared global part store was introduced
Rejected: Keep generic passives as the default style | repeated verification failures from upstream EasyEDA API instability
Rejected: Add ad hoc offline hacks around ato part-picking | weaker than making the package source deterministic
Confidence: high
Scope-risk: moderate
Reversibility: clean
Directive: For packages that already own generated local parts, instantiate those part modules directly and avoid generic passive declarations unless there is a strong reason not to
Tested:  passed for stm32g0b1kbu6_st, mcp2518fdt_e_sl_microchip, tcan3413ddfr_ti, raspberry_pi_hat_socket_zhouri, bq40z50rsmr_r2_4s_3a_ti, tps56637rpar_5v1_5a_ti, tps62933drlr_3v3_ti, bq25756rrvr_4s_2a_ti, tps2121ruxr_20v_4a_ti, and tps25730drefr_20v_3a_ti
Not-tested: Cross-package downstream integration beyond each package's default/example build
Parts:
- C1, C14, C15, C16, C2, C3, C4, C5, C6, C7, C8, C9: value 0F -> (none)
- L1: value L 0H -> (none)
- R1, R6: value 0.005Ω -> (none)
- R10: value 249000Ω -> (none)
- R13, R2: value 49900Ω -> (none)
- R14, R15, R3: value 10000Ω -> (none)
- R4, R5, R7, R8: value 10Ω -> (none)
- R9: value 24900Ω -> (none)
Connections:
- net battery_bulk_pack-power-hv renamed battery-hv
- net battery_bypass-power-hv renamed 1-1
- net battery_sense_filter-power-hv renamed srp_filtered
- net battery_sense_filter-power-lv renamed srn_filtered
- net bootstrap_1-power-hv renamed 1-2
- net bootstrap_1-power-lv renamed 1-3
- net bootstrap_2-power-hv renamed 1-4
- net regn_bulk-power-hv renamed 1-5
- net vac_bypass-power-hv renamed 1
- C1 pad 1: hv -> acp_filtered
- C1 pad 2: lv -> acn_filtered
- C14 pad 2: vac_bypass-power-lv -> lv
- C15 pad 2: vac_bypass-power-lv -> lv
- C16 pad 2: vac_bypass-power-lv -> lv
- C2 pad 2: vac_bypass-power-lv -> lv
- C3 pad 2: vac_bypass-power-lv -> lv
- C4 pad 2: vac_bypass-power-lv -> lv
- C5 pad 1: input_bulk_source-power-hv -> hv
- C5 pad 2: vac_bypass-power-lv -> lv
- C6 pad 2: vac_bypass-power-lv -> lv
- C9 pad 2: bootstrap_2-power-lv -> 2
- L1 pad 2: bootstrap_2-power-lv -> 2
- Q1 pad 1: bootstrap_2-power-lv -> 2
- Q1 pad 3: vac_bypass-power-lv -> lv
- Q1 pad 5: bootstrap_2-power-lv -> 2
- Q2 pad 2: 2 -> 2-1
- Q2 pad 3: vac_bypass-power-lv -> lv
- R13 pad 2: vac_bypass-power-lv -> lv
- R14 pad 2: vac_bypass-power-lv -> lv
- R2 pad 2: vac_bypass-power-lv -> lv
- R3 pad 2: vac_bypass-power-lv -> lv
- R4 pad 2: lv -> acn_filtered
- R5 pad 1: input_bulk_source-power-hv -> hv
- R5 pad 2: hv -> acp_filtered
- R6 pad 1: input_bulk_source-power-hv -> hv
- R9 pad 2: vac_bypass-power-lv -> lv
- U1 pad 10: vac_bypass-power-lv -> lv
- U1 pad 11: vac_bypass-power-lv -> lv
- U1 pad 17: vac_bypass-power-lv -> lv
- U1 pad 18: bootstrap_2-power-lv -> 2
- U1 pad 22: vac_bypass-power-lv -> lv
- U1 pad 27: 2 -> 2-1
- U1 pad 29: lv -> acn_filtered
- U1 pad 30: hv -> acp_filtered
- U1 pad 35: vac_bypass-power-lv -> lv
- U1 pad 37: vac_bypass-power-lv -> lv

Commit message: Make package schematics more readable and align passive choices with repo guidance
This pass improves the human-facing quality of the package library.
Explicit local capacitor/resistor parts now carry short descriptive
comments at the point of use, the MCP2518FD package swaps its 1uF bulk
capacitor to a 0603 part to match the current sizing rule, and several
packages add better net-name overrides for exposed and important internal
signals.

Constraint: Repo guidance now prefers explicit local parts and expects readable schematic net names
Constraint: Passive sizing should follow the current MLCC package rule unless a justified exception is needed
Rejected: Keep part instances comment-free | explicit local part names are not readable enough by themselves
Rejected: Leave the MCP2518FD 1uF bulk cap in 0402 | conflicts with the current 1uF-10uF 0603 guidance
Confidence: medium
Scope-risk: moderate
Reversibility: clean
Directive: When instantiating explicit local resistor/capacitor parts, include a short readable comment with the key value/package characteristics unless the name is already obviously human-readable
Tested:  passed for stm32g0b1kbu6_st, mcp2518fdt_e_sl_microchip, tcan3413ddfr_ti, raspberry_pi_hat_socket_zhouri, bq40z50rsmr_r2_4s_3a_ti, tps56637rpar_5v1_5a_ti, tps62933drlr_3v3_ti, bq25756rrvr_4s_2a_ti, tps2121ruxr_20v_4a_ti, and tps25730drefr_20v_3a_ti
Not-tested: Complete elimination of all internal autogenerated net labels in every package; some deep internal nets may still remain tool-driven
Connections:
- net 1 renamed INPUT_BUS
- net 1-1 renamed CHARGE_BUS
- net 1-2 renamed BTST1
- net 1-3 renamed SW1
- net 1-4 renamed BTST2
- net 1-5 renamed REGN
- net 19 renamed HIDRV2
- net 2 renamed SW2
- net 2-1 renamed HIDRV1
- net 21 renamed LODRV2
- net 25 renamed LODRV1
- net 4 renamed STAT1
- net 5 renamed STAT2
- net acn_filtered renamed ACN_FILT
- net acp_filtered renamed ACP_FILT
- net lv renamed GND
- net srn_filtered renamed SRN_FILT
- net srp_filtered renamed SRP_FILT

Commit message: Finish removing net-name overrides from reusable packages
This completes the package-level override cleanup by deleting the remaining
`override_net_name` assignments from the library's reusable package modules and
rebuilding their checked-in layouts so generated net metadata matches source.
The package interfaces stay the same; only the forced net naming was removed so
these modules compose cleanly when imported into downstream designs.

Constraint: The library must stay reusable and avoid imposed internal net names leaking into consuming designs
Constraint: Each changed package must still verify with the repo's Atopile workflow after layout regeneration
Rejected: Stop after the battery frontend cleanup | leaves the same composition hazard in other packages
Rejected: Remove override lines without rebuilding layouts | would leave stale generated PCB net names checked into the repo
Confidence: high
Scope-risk: moderate
Reversibility: clean
Directive: Do not reintroduce `override_net_name` in reusable package modules unless a package is intentionally design-specific
Tested: `uv tool run --from atopile==0.15.4 ato --non-interactive build` in each affected package directory (stm32g0b1kbu6_st, mcp2518fdt_e_sl_microchip, tcan3413ddfr_ti, raspberry_pi_hat_socket_zhouri, tps56637rpar_5v1_5a_ti, tps62933drlr_3v3_ti, bq25756rrvr_4s_2a_ti, tps2121ruxr_20v_4a_ti, tps25730drefr_20v_3a_ti)
Not-tested: Downstream consumer projects that may have been depending on the old forced net names in generated layouts
Connections:
- net ACN_FILT renamed acn_filtered
- net ACP_FILT renamed acp_filtered
- net BTST1 renamed 1-2
- net BTST2 renamed 1-4
- net CHARGE_BUS renamed 1-1
- net GND renamed lv
- net HIDRV1 renamed 2-1
- net HIDRV2 renamed 19
- net INPUT_BUS renamed 1
- net LODRV1 renamed 25
- net LODRV2 renamed 21
- net REGN renamed 1-5
- net SRN_FILT renamed srn_filtered
- net SRP_FILT renamed srp_filtered
- net STAT1 renamed 4
- net STAT2 renamed 5
- net SW1 renamed 1-3
- net SW2 renamed 2

Commit message: Reduce BQ25756 feedback divider footprint without changing regulation
The charger package used a 0603 249 kΩ / 0.1% FB-top resistor even though the
node's dissipation and voltage stress allow a 0402 part. This swaps in a
concrete 0402 Viking Tech resistor with the same nominal value and tolerance so
layout stays tighter without changing the programmed charge voltage.

Constraint: Keep the exact 249 kΩ / 0.1% feedback ratio to preserve standalone charge-voltage programming
Constraint: Must use an LCSC-sourced deterministic part compatible with local Atopile assets
Rejected: Relax the FB divider to 1% parts | unnecessary hit to regulation accuracy budget
Rejected: Recalculate the divider around a different readily-available value | no functional need when an exact 0402 option exists
Confidence: high
Scope-risk: narrow
Reversibility: clean
Directive: Keep the FB top resistor at 249 kΩ 0.1% unless the charge-voltage target and accuracy budget are re-derived together
Tested:  in packages/power/charger/bq25756rrvr_4s_2a_ti (default and example)
Not-tested: Hardware-level charge-voltage tolerance across resistor/process/temperature variation
Parts:
- R10: footprint YAGEO_RT0603BRD07249KL:R0603 -> Viking_Tech_ARG02BTC2493:R0402
Changed lines of the file:
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@@
 		)
 	)
-	(footprint "YAGEO_RT0603BRD07249KL:R0603"
+	(footprint "Viking_Tech_ARG02BTC2493:R0402"
 		(layer "F.Cu")
 		(at 30 -290 0)
@@
 			)
 		)
-		(property "LCSC" "C705752"
+		(property "LCSC" "C2984416"
 			(at 0 0 0)
 			(layer "User.9")
 			(hide yes)
 		)
-		(property "Manufacturer" "YAGEO"
+		(property "Manufacturer" "Viking Tech"
 			(at 0 0 0)
 			(layer "User.9")
@@
 			(hide yes)
 		)
-		(property "Partnumber" "RT0603BRD07249KL"
+		(property "Partnumber" "ARG02BTC2493"
 			(at 0 0 0)
 			(layer "User.9")
 			(hide yes)
 		)
-		(property "Datasheet" "https://wmsc.lcsc.com/wmsc/upload/file/pdf/v2/lcsc/2009282205_YAGEO-RT0603BRD07249KL_C705752.pdf"
+		(property "Datasheet" "https://wmsc.lcsc.com/wmsc/upload/file/pdf/v2/lcsc/2208081100_Viking-Tech-ARG02BTC2493_C2984416.pdf"
 			(at 0 0 0)
 			(layer "User.9")
@@
 			(hide yes)
 		)
-		(property "lcsc_id" "C705752"
+		(property "lcsc_id" "C2984416"
 			(at 0 0 0)
 			(layer "User.9")
@@
 			(hide yes)
 		)
-		(attr smd)
+		(attr through_hole)
 		(fp_line
-			(start 0.43 0.66)
-			(end 1.39 0.66)
+			(start -0.23 0.5)
+			(end -0.94 0.5)
 			(stroke
 				(width 0.15)
@@
 		)
 		(fp_line
-			(start 1.39 0.66)
-			(end 1.39 -0.66)
+			(start -0.94 0.5)
+			(end -0.94 -0.5)
 			(stroke
 				(width 0.15)
@@
 		)
 		(fp_line
-			(start 1.39 -0.66)
-			(end 0.43 -0.66)
+			(start -0.94 -0.5)
+			(end -0.23 -0.5)
 			(stroke
 				(width 0.15)
@@
 		)
 		(fp_line
-			(start -0.43 0.66)
-			(end -1.39 0.66)
+			(start 0.23 0.5)
+			(end 0.94 0.5)
 			(stroke
 				(width 0.15)
@@
 		)
 		(fp_line
-			(start -1.39 0.66)
-			(end -1.39 -0.66)
+			(start 0.94 0.5)
+			(end 0.94 -0.5)
 			(stroke
 				(width 0.15)
@@
 		)
 		(fp_line
-			(start -1.39 -0.66)
-			(end -0.43 -0.66)
+			(start 0.94 -0.5)
+			(end 0.23 -0.5)
 			(stroke
 				(width 0.15)
@@
 		)
 		(fp_circle
-			(center -0.8 0.4)
-			(end -0.77 0.4)
+			(center -0.5 0.25)
+			(end -0.47 0.25)
 			(stroke
 				(width 0.06)
@@
 		)
 		(pad "2" smd rect
-			(at 0.75 0 0)
-			(size 0.81 0.86)
+			(at 0.43 0 0)
+			(size 0.57 0.54)
 			(layers "F.Cu" "F.Paste" "F.Mask")
 			(net 24 "FB")
 		)
 		(pad "1" smd rect
-			(at -0.75 0 0)
-			(size 0.81 0.86)
+			(at -0.43 0 0)
+			(size 0.57 0.54)
 			(layers "F.Cu" "F.Paste" "F.Mask")
 			(net 30 "battery-hv")
 		)
 		(embedded_fonts no)
-		(model "${KIPRJMOD}/../../parts/YAGEO_RT0603BRD07249KL/R0603.STEP"
+		(model "${KIPRJMOD}/../../parts/Viking_Tech_ARG02BTC2493/R0402_L1.0-W0.5-H0.4.step"
 			(offset
-				(xyz 0 0 -0)
+				(xyz 0 -0 0)
 			)
 			(scale
@@
 			)
 			(rotate
-				(xyz 0 0 270)
+				(xyz 0 0 0)
 			)
 		)

Commit message: charger layout
Parts:
- removed C14, C6: , Murata_Electronics_GRM155R71H104KE14D:C0402
- added C10: , Murata_Electronics_GRM31CR71H475KA12L:C1206, F.Cu at (80.9, 42.2)
- added C11: , Murata_Electronics_GRM155R71H104KE14D:C0402, F.Cu at (81.6, 44.0)
- added C12: , Murata_Electronics_GRM31CR71H475KA12L:C1206, F.Cu at (67.1, 42.2)
- added C13: , Murata_Electronics_GRM155R71H104KE14D:C0402, F.Cu at (66.4, 44.0)
- added Q3: , Texas_Instruments_CSD18543Q3A:VSONP-8_L3.1-W3.1-P0.65-LS3.5-BL, F.Cu at (63.7, 46.6)
- added Q4: , Texas_Instruments_CSD18543Q3A:VSONP-8_L3.1-W3.1-P0.65-LS3.5-BL, F.Cu at (68.0, 46.7)
- C15: footprint Murata_Electronics_GRM31CR71H475KA12L:C1206 -> Murata_Electronics_GRM188R61E475KE11D:C0603
- Q1, Q2: footprint XNRUSEMI_XRS30V06D:DFN-8_L3.3-W3.3-P0.75-TL -> Texas_Instruments_CSD18543Q3A:VSONP-8_L3.1-W3.1-P0.65-LS3.5-BL
- moved C16 368.1 mm to (68.5, 56.1), turned to 180 degrees
- moved R13 360.3 mm to (68.9, 58.2), turned to 180 degrees
- moved R10 351.1 mm to (80.1, 57.5), turned to 180 degrees
- moved C15 333.7 mm to (73.9, 50.8), turned to -90 degrees
- moved L1 318.0 mm to (74.0, 44.9)
- moved R15 284.0 mm to (75.5, 60.3), turned to 90 degrees
- moved R14 274.3 mm to (76.7, 60.3), turned to -90 degrees
- moved R3 205.1 mm to (74.3, 60.3), turned to -90 degrees
- moved R9 195.2 mm to (80.1, 58.7)
- moved R2 186.6 mm to (77.9, 60.3), turned to -90 degrees
- moved R6 148.1 mm to (64.5, 34.0), turned to -90 degrees
- moved R1 144.3 mm to (83.5, 34.0), turned to 90 degrees
- moved C9 138.1 mm to (75.7, 50.3), turned to 90 degrees
- moved C8 127.5 mm to (72.1, 50.3), turned to 90 degrees
- moved R8 116.9 mm to (80.1, 55.1), turned to 180 degrees
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Connections:
- C15 pad 1: 1-5 -> lv
- C15 pad 2: lv -> 1-5
- Q1 pad 2: 19 -> 2
- Q1 pad 3: lv -> 2
- Q1 pad 4: 21 -> G
- Q1 pad 5: 2 -> 1-1
- Q2 pad 1: 1-3 -> lv
- Q2 pad 2: 2-1 -> lv
- Q2 pad 4: 25 -> G-1
- Q2 pad 5: 1-3 -> 2
- Q2 pad 8: 1 -> 2
- U1 pad 19: 19 -> G
- U1 pad 21: 21 -> G-1
- U1 pad 25: 25 -> G-3
- U1 pad 27: 2-1 -> G-2
Routing:
- net battery-hv: track 0.00 -> 56.3 mm, vias 0 -> 4
- net 1: track 0.00 -> 36.8 mm, vias 0 -> 4
- net 1-1: track 0.00 -> 25.2 mm, vias 0 -> 2
- net hv: track 0.00 -> 24.0 mm, vias 0 -> 2
- net 1-3: track 0.00 -> 12.1 mm, vias 0 -> 2
- net 2: track 0.00 -> 12.0 mm, vias 0 -> 2
- net G-3: track 0.00 -> 11.8 mm, vias 0 -> 2
- net G-2: track 0.00 -> 11.4 mm, vias 0 -> 2
- net G-1: track 0.00 -> 10.1 mm, vias 0 -> 2
- net G: track 0.00 -> 10.1 mm, vias 0 -> 2
- net 1-5: track 0.00 -> 10.0 mm, vias 0 -> 2
- net FB: track 0.00 -> 4.16 mm
- net ICHG: track 0.00 -> 3.38 mm
- net srp_filtered: track 0.00 -> 3.16 mm
- net acn_filtered: track 0.00 -> 3.08 mm
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- added copper zone on F.Cu, net 1
- added copper zone on F.Cu, net 1-1
- added copper zone on F.Cu, net 1-3
- added copper zone on F.Cu, net 1-5
- added copper zone on F.Cu, net 2
- added copper zone on F.Cu, net battery-hv
- added copper zone on F.Cu, net hv
Other:
- copper layers 2 -> 4
