File: packages/power/battery_management/bq40z50rsmr_r2_4s_3a_ti/layouts/default/default.kicad_pcb (KiCad board)
At the start: 2 copper layers, 25 parts

Commit message: 22uF cap update, TPS56637 update
Parts:
- C1, C4, C5, C6, C7: footprint Murata_Electronics_GRM155R71E104KE14D:C0402 -> Murata_Electronics_GRM155R71H104KE14D:C0402
Changed lines of the file:
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@@
 		)
 	)
-	(footprint "Murata_Electronics_GRM155R71E104KE14D:C0402"
+	(footprint "Murata_Electronics_GRM155R71H104KE14D:C0402"
 		(layer "F.Cu")
 		(at 20 -170 0)
@@
 			)
 		)
-		(property "LCSC" "C77014"
+		(property "LCSC" "C77020"
 			(at 0 0 0)
 			(layer "User.9")
@@
 			(hide yes)
 		)
-		(property "Partnumber" "GRM155R71E104KE14D"
-			(at 0 0 0)
-			(layer "User.9")
-			(hide yes)
-		)
-		(property "Datasheet" "https://www.lcsc.com/datasheet/lcsc_datasheet_1811081616_Murata-Electronics-GRM155R71E104KE14D_C77014.pdf"
+		(property "Partnumber" "GRM155R71H104KE14D"
+			(at 0 0 0)
+			(layer "User.9")
+			(hide yes)
+		)
+		(property "Datasheet" "https://www.lcsc.com/datasheet/lcsc_datasheet_1809272047_Murata-Electronics-GRM155R71H104KE14D_C77020.pdf"
 			(at 0 0 0)
 			(layer "User.9")
@@
 			(hide yes)
 		)
-		(property "lcsc_id" "C77014"
+		(property "lcsc_id" "C77020"
 			(at 0 0 0)
 			(layer "User.9")
@@
 		)
 		(embedded_fonts no)
-		(model "${KIPRJMOD}/../../parts/Murata_Electronics_GRM155R71E104KE14D/C0402_L1.0-W0.5-H0.5.step"
+		(model "${KIPRJMOD}/../../parts/Murata_Electronics_GRM155R71H104KE14D/C0402_L1.0-W0.5-H0.5.step"
 			(offset
 				(xyz 0 0 -0)
@@
 		)
 	)
-	(footprint "Murata_Electronics_GRM155R71E104KE14D:C0402"
+	(footprint "Murata_Electronics_GRM155R71H104KE14D:C0402"
 		(layer "F.Cu")
 		(at 20 -180 0)
@@
 			)
 		)
-		(property "LCSC" "C77014"
+		(property "LCSC" "C77020"
 			(at 0 0 0)
 			(layer "User.9")
@@
 			(hide yes)
 		)
-		(property "Partnumber" "GRM155R71E104KE14D"
-			(at 0 0 0)
-			(layer "User.9")
-			(hide yes)
-		)
-		(property "Datasheet" "https://www.lcsc.com/datasheet/lcsc_datasheet_1811081616_Murata-Electronics-GRM155R71E104KE14D_C77014.pdf"
+		(property "Partnumber" "GRM155R71H104KE14D"
+			(at 0 0 0)
+			(layer "User.9")
+			(hide yes)
+		)
+		(property "Datasheet" "https://www.lcsc.com/datasheet/lcsc_datasheet_1809272047_Murata-Electronics-GRM155R71H104KE14D_C77020.pdf"
 			(at 0 0 0)
 			(layer "User.9")
@@
 			(hide yes)
 		)
-		(property "lcsc_id" "C77014"
+		(property "lcsc_id" "C77020"
 			(at 0 0 0)
 			(layer "User.9")
@@
 		)
 		(embedded_fonts no)
-		(model "${KIPRJMOD}/../../parts/Murata_Electronics_GRM155R71E104KE14D/C0402_L1.0-W0.5-H0.5.step"
+		(model "${KIPRJMOD}/../../parts/Murata_Electronics_GRM155R71H104KE14D/C0402_L1.0-W0.5-H0.5.step"
 			(offset
 				(xyz 0 0 -0)
@@
 		)
 	)
-	(footprint "Murata_Electronics_GRM155R71E104KE14D:C0402"
+	(footprint "Murata_Electronics_GRM155R71H104KE14D:C0402"
 		(layer "F.Cu")
 		(at 20 -190 0)
@@
 			)
 		)
-		(property "LCSC" "C77014"
+		(property "LCSC" "C77020"
 			(at 0 0 0)
 			(layer "User.9")
@@
 			(hide yes)
 		)
-		(property "Partnumber" "GRM155R71E104KE14D"
-			(at 0 0 0)
-			(layer "User.9")
-			(hide yes)
-		)
-		(property "Datasheet" "https://www.lcsc.com/datasheet/lcsc_datasheet_1811081616_Murata-Electronics-GRM155R71E104KE14D_C77014.pdf"
+		(property "Partnumber" "GRM155R71H104KE14D"
+			(at 0 0 0)
+			(layer "User.9")
+			(hide yes)
+		)
+		(property "Datasheet" "https://www.lcsc.com/datasheet/lcsc_datasheet_1809272047_Murata-Electronics-GRM155R71H104KE14D_C77020.pdf"
 			(at 0 0 0)
 			(layer "User.9")
@@
 			(hide yes)
 		)
-		(property "lcsc_id" "C77014"
+		(property "lcsc_id" "C77020"
 			(at 0 0 0)
 			(layer "User.9")
@@
 		)
 		(embedded_fonts no)
-		(model "${KIPRJMOD}/../../parts/Murata_Electronics_GRM155R71E104KE14D/C0402_L1.0-W0.5-H0.5.step"
+		(model "${KIPRJMOD}/../../parts/Murata_Electronics_GRM155R71H104KE14D/C0402_L1.0-W0.5-H0.5.step"
 			(offset
 				(xyz 0 0 -0)
@@
 		)
 	)
-	(footprint "Murata_Electronics_GRM155R71E104KE14D:C0402"
+	(footprint "Murata_Electronics_GRM155R71H104KE14D:C0402"
 		(layer "F.Cu")
 		(at 20 -200 0)
@@
 			)
 		)
-		(property "LCSC" "C77014"
+		(property "LCSC" "C77020"
 			(at 0 0 0)
 			(layer "User.9")
@@
 			(hide yes)
 		)
-		(property "Partnumber" "GRM155R71E104KE14D"
-			(at 0 0 0)
-			(layer "User.9")
-			(hide yes)
-		)
-		(property "Datasheet" "https://www.lcsc.com/datasheet/lcsc_datasheet_1811081616_Murata-Electronics-GRM155R71E104KE14D_C77014.pdf"
+		(property "Partnumber" "GRM155R71H104KE14D"
+			(at 0 0 0)
+			(layer "User.9")
+			(hide yes)
+		)
+		(property "Datasheet" "https://www.lcsc.com/datasheet/lcsc_datasheet_1809272047_Murata-Electronics-GRM155R71H104KE14D_C77020.pdf"
 			(at 0 0 0)
 			(layer "User.9")
@@
 			(hide yes)
 		)
-		(property "lcsc_id" "C77014"
+		(property "lcsc_id" "C77020"
 			(at 0 0 0)
 			(layer "User.9")
@@
 		)
 		(embedded_fonts no)
-		(model "${KIPRJMOD}/../../parts/Murata_Electronics_GRM155R71E104KE14D/C0402_L1.0-W0.5-H0.5.step"
+		(model "${KIPRJMOD}/../../parts/Murata_Electronics_GRM155R71H104KE14D/C0402_L1.0-W0.5-H0.5.step"
 			(offset
 				(xyz 0 0 -0)
@@
 		)
 	)
-	(footprint "Murata_Electronics_GRM155R71E104KE14D:C0402"
+	(footprint "Murata_Electronics_GRM155R71H104KE14D:C0402"
 		(layer "F.Cu")
 		(at 0 0 0)
@@
 			)
 		)
-		(property "LCSC" "C77014"
+		(property "LCSC" "C77020"
 			(at 0 0 0)
 			(layer "User.9")
@@
 			(hide yes)
 		)
-		(property "Partnumber" "GRM155R71E104KE14D"
-			(at 0 0 0)
-			(layer "User.9")
-			(hide yes)
-		)
-		(property "Datasheet" "https://www.lcsc.com/datasheet/lcsc_datasheet_1811081616_Murata-Electronics-GRM155R71E104KE14D_C77014.pdf"
+		(property "Partnumber" "GRM155R71H104KE14D"
+			(at 0 0 0)
+			(layer "User.9")
+			(hide yes)
+		)
+		(property "Datasheet" "https://www.lcsc.com/datasheet/lcsc_datasheet_1809272047_Murata-Electronics-GRM155R71H104KE14D_C77020.pdf"
 			(at 0 0 0)
 			(layer "User.9")
@@
 			(hide yes)
 		)
-		(property "lcsc_id" "C77014"
+		(property "lcsc_id" "C77020"
 			(at 0 0 0)
 			(layer "User.9")
@@
 		)
 		(embedded_fonts no)
-		(model "${KIPRJMOD}/../../parts/Murata_Electronics_GRM155R71E104KE14D/C0402_L1.0-W0.5-H0.5.step"
+		(model "${KIPRJMOD}/../../parts/Murata_Electronics_GRM155R71H104KE14D/C0402_L1.0-W0.5-H0.5.step"
 			(offset
 				(xyz 0 0 -0)

Commit message: wip
Parts:
- added Q2: , Texas_Instruments_CSD18543Q3A:VSONP-8_L3.1-W3.1-P0.65-LS3.5-BL, F.Cu at (80.2, 60.2)
- Q1: footprint XNRUSEMI_XRS30V06D:DFN-8_L3.3-W3.3-P0.75-TL -> Texas_Instruments_CSD18543Q3A:VSONP-8_L3.1-W3.1-P0.65-LS3.5-BL
- moved C7 243.0 mm to (61.1, 39.5), turned to -90 degrees
- moved C6 234.9 mm to (61.1, 41.3), turned to -90 degrees
- moved C5 227.0 mm to (61.1, 43.2), turned to -90 degrees
- moved C4 209.4 mm to (60.3, 35.5), turned to 180 degrees
- moved R13 202.9 mm to (59.6, 39.0)
- moved R12 195.4 mm to (59.6, 41.3)
- moved R11 186.7 mm to (59.6, 42.5)
- moved R10 178.2 mm to (59.6, 43.7)
- moved R9 176.8 mm to (60.3, 52.1), turned to 90 degrees
- moved R8 166.5 mm to (57.1, 52.3), turned to 90 degrees
- moved R7 159.3 mm to (58.8, 54.5)
- moved C8 146.0 mm to (65.7, 35.0), turned to 180 degrees
- moved R4 138.1 mm to (81.2, 63.8)
- moved R2 126.0 mm to (73.6, 64.0)
- moved R3 122.5 mm to (80.9, 66.3)
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Connections:
- C1 pad 1: 1-1 -> 1
- C8 pad 1: 1-2 -> 1-1
- Q1 pad 1: raw_battery-hv -> hv
- Q1 pad 2: 2 -> hv
- Q1 pad 4: 1 -> G
- Q1 pad 5: fet_common -> D
- Q1 pad 8: fet_common -> D
- R1 pad 1: 1 -> G
- R2 pad 2: 1 -> G
- R3 pad 1: 2 -> G-1
- R4 pad 2: 2 -> G-1
- R5 pad 1: 1-1 -> 1
- U1 pad 1: 1-2 -> 1-1
- U1 pad 23: 1-1 -> 1
